File: PCBs/Motor Controller Board/RP2040_minimal_r2/_autosave-RP2040_minimal_r2.kicad_sch (KiCad schematic)
At the start: 34 parts, among them J1 USB_B_Micro, J2 Conn_01x02, J3 Conn_02x18_Odd_Even, J4 Conn_02x18_Odd_Even, U1 NCP1117-3.3_SOT223, U2 W25Q128JVS, U3 RP2040, Y1 ABM8-272-T3

Commit message: vault backup: 2025-04-07 16:10:55
Parts:
- added J5: Conn_01x06_MountingPin, symbol Connector_Generic_MountingPin:Conn_01x06_MountingPin
- added U4: DRV8243HQDGQRQ1, HVSSOP28_DGQ_TEX, symbol New_Library:DRV8243HQDGQRQ1
Connections:
- net GND: now also U4.12 (GND), U4.13 (GND), U4.14 (GND), U4.15 (GND), U4.16 (GND), U4.17 (GND), U4.29 (GND)
- new net: J5.2 (Pin_2), U4.10 (OUT1), U4.11 (OUT1), U4.9 (OUT1)
- new net: J5.1 (Pin_1), U4.18 (OUT2), U4.19 (OUT2), U4.20 (OUT2)

Commit message: vault backup: 2025-04-07 16:42:59
Parts:
- added J6: Conn_01x02, symbol Connector_Generic:Conn_01x02
- added R6, R7: 100k, symbol Device:R
Connections:
- net GND: now also J5.3 (Pin_3), J6.1 (Pin_1), R6.1, R7.1
- net VBUS: now also J5.4 (Pin_4)
- net at U4.1 (SR): now also R7.2
- net at U4.2 (DIAG): now also R6.2
- net VM: now reaches U4.21 (VM)
- net VM: now also U4.22 (VM), U4.23 (VM), U4.6 (VM), U4.7 (VM), U4.8 (VM), J6.2 (Pin_2)
- net EncA: now reaches J5.5 (Pin_5)
- net EncB: now reaches J5.6 (Pin_6)
Other:
- moved on the sheet: C17, J3, J4, J5, U4
