File: PCBs/ModuleBoard/RP2040_minimal_r2/_autosave-SwerveModuleBoard.kicad_pcb (KiCad board)
At the start: 2 copper layers, 52 parts, among them J1 USB_B_Micro, J2 Conn_01x02, J4 Conn_01x07, J5 Conn_01x06_Pin, J6 Conn_01x02, J7 Conn_01x06_Pin, J8 Conn_01x06, U1 NCP1117-3.3_SOT223, U2 W25Q128JVS, U3 RP2040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

Commit message: vault backup: 2025-04-24 00:37:27
Parts:
- removed J2: Conn_01x02, Connector_PinHeader_2.54mm:PinHeader_1x02_P2.54mm_Vertical
- moved H3 77.7 mm to (125.0, 117.8)
- moved H1 65.3 mm to (75.0, 117.8)
- moved H2 60.8 mm to (118.4, 73.6)
- moved U2 58.3 mm to (77.5, 31.0)
- moved C17 58.3 mm to (81.5, 24.2)
- moved C5 58.3 mm to (80.7, 26.6)
- moved R1 58.3 mm to (75.5, 26.1)
- moved R2 58.3 mm to (74.0, 26.1)
- moved H4 43.8 mm to (81.6, 73.6)
- moved BTSEL1 6.25 mm to (77.8, 89.8)
Routing:
- net /QSPI_SS: track 22.6 -> 4.61 mm
- net /QSPI_SD1: track 16.8 -> 1.71 mm
- net /QSPI_SD2: track 13.1 -> 2.32 mm
- net /QSPI_SD3: track 13.2 -> 3.78 mm
- net /QSPI_SCLK: track 11.6 -> 2.34 mm
- net /QSPI_SD0: track 9.08 -> 0.00 mm
- net +3V3: track 227.9 -> 219.7 mm
- net /~{USB_BOOT}: track 5.34 -> 0.00 mm
Other:
- board outline added: 60 x 52.9 mm

Commit message: vault backup: 2025-04-24 00:52:44
Parts:
- moved C18 15.8 mm to (111.9, 137.2)
- moved C20 15.8 mm to (92.2, 137.2)
- moved C21 15.8 mm to (106.2, 139.4)
- moved J5 15.8 mm to (75.8, 148.2)
- moved J6 15.8 mm to (97.9, 149.2)
- moved J7 15.8 mm to (123.5, 148.2)
- moved R6 15.8 mm to (83.3, 132.4)
- moved R7 15.8 mm to (80.6, 134.3)
- moved R9 15.8 mm to (119.9, 133.7)
- moved U4 15.8 mm to (83.9, 140.1)
- moved U5 15.8 mm to (119.5, 140.0)
- moved C19 15.8 mm to (98.7, 139.4)
- moved J4 12.1 mm to (141.8, 103.2)
- moved J8 8.84 mm to (58.5, 92.2)
- moved C10 7.60 mm to (102.8, 86.8)
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Routing:
- net +3V3: track 219.7 -> 111.9 mm, vias 2 -> 3
- net /GPIO6: track 99.6 -> 0.00 mm
- net /GPIO7: track 95.6 -> 0.00 mm
- net /GPIO8: track 42.0 -> 0.00 mm
- net /GPIO9: track 41.5 -> 0.00 mm
- net /GPIO5: track 35.0 -> 0.00 mm
- net /GPIO4: track 34.0 -> 0.00 mm
- net /GPIO23: track 33.7 -> 0.00 mm
- net /GPIO3: track 33.1 -> 0.00 mm
- net /GPIO24: track 32.8 -> 0.00 mm
- net /GPIO2: track 32.2 -> 0.00 mm
- net /GPIO25: track 31.9 -> 0.00 mm
- net /GPIO20: track 31.5 -> 0.00 mm
- net /GPIO10: track 31.4 -> 0.00 mm
- net /GPIO1: track 31.3 -> 0.00 mm
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