File: PCBs/ModuleBoard/RP2040_minimal_r2/_autosave-SwerveModuleBoard.kicad_pcb (KiCad board)
At the start: 2 copper layers, 60 x 52.9 mm, 57 parts, among them IC1 AS5600-ASOT, J1 USB_B_Micro, J3 Conn_02x08_Odd_Even_MountingP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, J4 Conn_01x07, J5 Conn_01x06_Pin, J6 Conn_01x02, J7 Conn_01x06_Pin, J8 Conn_01x06, U2 W25Q128JVS, U3 RP2040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

Commit message: vault backup: 2025-04-25 02:22:44
Parts:
- moved R9 37.5 mm to (114.5, 96.5), turned to 90 degrees
- moved R10 2.15 mm to (108.8, 99.2)
- moved D1 0.52 mm to (106.9, 97.5)
Routing:
- net VM: track 51.4 -> 83.2 mm
- net /GPIO19: track 0.00 -> 24.8 mm
- net /GPIO20: track 0.00 -> 23.4 mm
- net /GPIO18: track 0.00 -> 23.2 mm
- net /GPIO17: track 11.3 -> 0.00 mm
- net +5V: track 76.6 -> 84.4 mm
- net +3V3: track 103.9 -> 98.7 mm
- net GND: track 121.7 -> 125.2 mm, vias 52 -> 55
- net Net-(U5-SR): track 2.87 -> 5.82 mm
- net Net-(D1-K): track 3.50 -> 1.79 mm

Commit message: vault backup: 2025-04-25 02:37:59
Parts:
- moved C21 34.6 mm to (120.2, 107.8)
- moved C22 31.9 mm to (104.5, 96.8)
- moved C18 29.5 mm to (125.0, 110.8), turned to 180 degrees
- moved R8 2.85 mm to (103.8, 101.5)
Routing:
- net +3V3: track 98.7 -> 136.1 mm, vias 2 -> 3
- net /GPIO16: track 0.00 -> 25.2 mm
- net /GPIO17: track 0.00 -> 22.3 mm
- net GND: track 125.2 -> 137.2 mm
- net /GPIO21: track 7.58 -> 8.44 mm
- net /GPIO20: track 23.4 -> 24.1 mm
- net /GPIO19: track 24.8 -> 24.2 mm

Commit message: vault backup: 2025-04-25 02:47:00
Parts:
- moved C18 22.6 mm to (119.8, 88.8), turned to -90 degrees
- moved J4 8.05 mm to (143.3, 80.2), turned to -90 degrees
Routing:
- net Net-(J7-Pin_5): track 39.0 -> 11.5 mm
- net GND: track 137.2 -> 111.7 mm, vias 55 -> 48
- net Net-(J7-Pin_6): track 34.6 -> 11.6 mm
- net VM: track 83.2 -> 74.2 mm
- net Net-(U5-SR): track 5.82 -> 2.94 mm
- net +1V1: track 26.1 -> 28.1 mm

Commit message: vault backup: 2025-04-25 02:57:11
Parts:
- moved J5 54.9 mm to (75.0, 93.2), turned to 0 degrees
- moved J8 20.8 mm to (60.0, 71.4)
Routing:
- net /GPIO3: track 0.00 -> 13.8 mm, vias 0 -> 1
- net /GPIO2: track 0.00 -> 12.9 mm, vias 0 -> 1
- net +3V3: track 136.2 -> 141.1 mm, vias 3 -> 4
- net +1V1: track 28.1 -> 31.3 mm
- added copper zone on B.Cu, net GND
