File: PCBs/ModuleBoard/RP2040_minimal_r2/_autosave-SwerveModuleBoard.kicad_pcb (KiCad board)
At the start: 2 copper layers, 60 x 52.9 mm, 57 parts, among them IC1 AS5600-ASOT, J1 USB_B_Micro, J3 Conn_02x08_Odd_Even_MountingP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, J4 Conn_01x07, J5 Conn_01x06_Pin, J6 Conn_01x02, J7 Conn_01x06_Pin, J8 Conn_01x06, U2 W25Q128JVS, U3 RP2040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

Commit message: vault backup: 2025-04-25 04:08:35
Parts:
- removed J8: Conn_01x06, Connector_PinHeader_2.54mm:PinHeader_1x06_P2.54mm_Vertical
- added J2: Conn_02x02_Counter_Clockwise, Connector_PinHeader_2.54mm:PinHeader_2x02_P2.54mm_Vertical, F.Cu at (84.8, 87.5)
- moved C13 3.00 mm to (86.8, 94.8)
Routing:
- net /GPIO6: track 0.00 -> 42.7 mm, vias 0 -> 2
- net /GPIO7: track 0.00 -> 40.0 mm, vias 0 -> 2
- net /GPIO0: track 0.00 -> 7.75 mm
- net /GPIO1: track 0.00 -> 6.53 mm
- net /GPIO2: track 14.4 -> 15.8 mm
- net /GPIO3: track 15.0 -> 15.8 mm

Commit message: vault backup: 2025-04-25 04:18:49
Parts:
- moved J2 3.65 mm to (81.2, 87.5), turned to 45 degrees
Connections:
- J2 pad 1: /GPIO1 -> GND
- J2 pad 3: GND -> /GPIO1
Routing:
- net +3V3: track 165.2 -> 174.4 mm
- net /GPIO1: track 6.53 -> 11.0 mm
- net VBUS: track 6.00 -> 3.09 mm
- net /GPIO0: track 7.75 -> 9.74 mm
- net /XIN: track 10.7 -> 12.0 mm
- net GND: track 95.1 -> 96.4 mm, vias 48 -> 49
- net /GPIO2: track 15.8 -> 14.8 mm
- removed copper zone on F.Cu, net VBUS
