File: PCBs/ModuleBoard/RP2040_minimal_r2/_autosave-SwerveModuleBoard.kicad_sch (KiCad schematic)
At the start: 52 parts, among them J1 USB_B_Micro, J2 Conn_02x08_Counter_Clockwise, J4 Conn_01x07, J5 Conn_01x06_Pin, J6 Conn_01x02, J7 Conn_01x06_Pin, J8 Conn_01x06, U1 NCP1117-3.3_SOT223, U2 W25Q128JVS, U3 RP2040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

Commit message: vault backup: 2025-04-24 02:13:32
Parts:
- added C22: 100n, symbol Device:C
- added IC1: AS5600-ASOT, AS5600-ASOT:SOIC127P600X175-8N, symbol AS5600-ASOT:AS5600-ASOT
Connections:
- net GND: now also C22.2, IC1.4 (GND)
- new net: C22.1, IC1.1 (VDD5V), IC1.2 (VDD3V3)
- no-connect marks 3 -> 5
