File: PCBs/ModuleBoard/RP2040_minimal_r2/SwerveModuleBoard.kicad_sch (KiCad schematic)
At the start: 60 parts, among them IC1 AS5600-ASOT, J1 USB_B_Micro, J3 Conn_02x08_Odd_Even_MountingP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, J4 Conn_01x07, J5 Conn_01x06_Pin, J6 Conn_01x02, J7 Conn_01x06_Pin, J8 Conn_01x06, U1 NCP1117-3.3_SOT223, U2 W25Q128JVS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

Commit message: vault backup: 2025-04-24 17:06:29
Parts:
- removed U6: TPS63051RMWR, RMW0012A, symbol TPS63051:TPS63051RMWR
- added U7: TPS63051RMWR, RMW0012A, symbol 2025-04-24_20-58-17:TPS63051RMWR
- U2: footprint Package_SO:SOIC-8_5.23x5.23mm_P1.27mm -> Package_SO:SOIC-8_5.3x5.3mm_P1.27mm
Connections:
- net +3V3: now also U7.4 (VOUT), U7.5 (FB)
- net GND: now also U7.2 (GND), U7.6 (PWM), U7.9 (GND)
- net VAA: now also U7.11 (EN), U7.12 (VIN)
- net at R12.2: now also U7.8 (PG)
- net at L2.1: now also U7.1 (L1)
- net at L2.2: now also U7.3 (L2)
- net at C26.1: now also U7.7 (SS)
Other:
- moved on the sheet: C1, C4, J1, U1

Commit message: vault backup: 2025-04-24 19:34:02
Parts:
- removed C1, C4: 10u, Capacitor_SMD:C_0603_1608Metric_Pad1.08x0.95mm_HandSolder, symbol Device:C
- removed U1: NCP1117-3.3_SOT223, Package_TO_SOT_SMD:SOT-223-3_TabPin2, symbol Regulator_Linear:NCP1117-3.3_SOT223
- added D3, D4: 1n4007, symbol Device:D
- U7: footprint RMW0012A -> BuckBoost:QFN50P250X250X100-12N
Connections:
- net VBUS: now also D3.2 (A)
- net VM: now also D4.2 (A)
- net VAA: no longer names the net of C25.1, U7.11 (EN), U7.12 (VIN)
- net VAA: now also D3.1 (K), D4.1 (K)

Commit message: vault backup: 2025-04-24 19:44:10
Parts:
- D3, D4: footprint (none) -> Diode_SMD:D_SOD-123
Changed lines of the file:
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@@
 			)
 		)
-		(property "Footprint" ""
+		(property "Footprint" "Diode_SMD:D_SOD-123"
 			(at 137.16 285.75 0)
 			(effects
@@
 			)
 		)
-		(property "Footprint" ""
+		(property "Footprint" "Diode_SMD:D_SOD-123"
 			(at 102.87 290.83 0)
 			(effects

Commit message: vault backup: 2025-04-25 01:51:37
Connections:
- net +5V: now reaches J3.14 (Pin_14)
- no-connect marks 6 -> 5
Changed lines of the file:
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@@
 		(at 213.36 255.27)
 	)
-	(no_connect
-		(at 49.53 146.05)
-	)
 	(wire
 		(pts
@@
 	(wire
 		(pts
+			(xy 54.61 146.05) (xy 54.61 151.13)
+		)
+		(stroke
+			(width 0)
+			(type default)
+		)
+	)
+	(wire
+		(pts
 			(xy 214.63 76.2) (xy 223.52 76.2)
 		)
@@
 	(wire
 		(pts
-			(xy 49.53 146.05) (xy 48.26 146.05)
+			(xy 48.26 146.05) (xy 54.61 146.05)
 		)
 		(stroke
@@
 	(wire
 		(pts
+			(xy 54.61 151.13) (xy 57.15 151.13)
+		)
+		(stroke
+			(width 0)
+			(type default)
+		)
+	)
+	(wire
+		(pts
 			(xy 120.65 27.94) (xy 118.11 27.94)
 		)
@@
 					(unit 1)
 				)
+			)
+		)
+	)
+	(symbol
+		(lib_id "power:+5V")
+		(at 57.15 151.13 0)
+		(unit 1)
+		(exclude_from_sim no)
+		(in_bom yes)
+		(on_board yes)
+		(dnp no)
+		(fields_autoplaced yes)
+		(property "Reference" "#PWR05"
+			(at 57.15 154.94 0)
+			(effects
+				(font
+					(size 1.27 1.27)
+				)
+				(hide yes)
+			)
+		)
+		(property "Value" "+5V"
+			(at 57.15 146.05 0)
+			(effects
+				(font
+					(size 1.27 1.27)
+				)
+			)
+		)
+		(property "Footprint" ""
+			(at 57.15 151.13 0)
+			(effects
+				(font
+					(size 1.27 1.27)
+				)
+				(hide yes)
+			)
+		)
+		(property "Datasheet" ""
+			(at 57.15 151.13 0)
+			(effects
+				(font
+					(size 1.27 1.27)
+				)
+				(hide yes)
+			)
+		)
+		(property "Description" "Power symbol creates a global label with name \"+5V\""
+			(at 57.15 151.13 0)
+			(effects
+				(font
+					(size 1.27 1.27)
+				)
+				(hide yes)
+			)
+		)
+		(pin "1"
+		)
+		(instances
+			(project ""
+				(path "/8c0b3d8b-46d3-4173-ab1e-a61765f77d61"
+					(reference "#PWR05")
+					(unit 1)
+				)

Commit message: AH BOARDS
Parts:
- removed C25, C27: 10μF, Capacitor_SMD:C_0603_1608Metric_Pad1.08x0.95mm_HandSolder, symbol Device:C
- removed C26: 1nF, Capacitor_SMD:C_0603_1608Metric_Pad1.08x0.95mm_HandSolder, symbol Device:C
- removed L2: 1.5 μH, Capacitor_SMD:C_0603_1608Metric_Pad1.08x0.95mm_HandSolder, symbol Device:L
- removed R12: 1M, Resistor_SMD:R_0603_1608Metric_Pad0.98x0.95mm_HandSolder, symbol Device:R
- removed U7: TPS63051RMWR, BuckBoost:QFN50P250X250X100-12N, symbol 2025-04-24_20-58-17:TPS63051RMWR
- added C23: 470 pF, Capacitor_SMD:C_0603_1608Metric, symbol Device:C
- added C24: 22 uF, Capacitor_SMD:C_1206_3216Metric_Pad1.33x1.80mm_HandSolder, symbol Device:C
- added D5, D6: PMEG3020EXEX, Diode_SMD:D_SOD-123F, symbol Device:D
- added R13: 10k, Resistor_SMD:R_0603_1608Metric, symbol Device:R
- added U6: MIC5219-3.3YM5, Package_TO_SOT_SMD:SOT-23-5, symbol Regulator_Linear:MIC5219-3.3YM5
Connections:
- net +3V3: now also C24.1, U6.5 (OUT)
- net +5V: now also D4.2 (A)
- net GND: now also C23.2, C24.2, U6.2 (GND)
- net VM: no longer D4.2 (A)
- new net: R13.1, U6.1 (IN)
- new net: R13.2, U6.3 (EN)
- new net: C23.1, U6.4 (BP)

Commit message: vault backup: 2025-04-25 02:02:09
Parts:
- removed D3, D4: 1n4007, Diode_SMD:D_SOD-123, symbol Device:D
Connections:
- net +5V: now also D5.2 (A)
- net VBUS: now also D6.2 (A)
- net at R13.1, U6.1 (IN): now also D5.1 (K), D6.1 (K)
Other:
- moved on the sheet: C23, C24, D5, D6, R13, U6

Commit message: vault backup: 2025-04-25 02:07:20
Connections:
- net at U5.5 (OUT2), U5.6 (OUT2): now also J7.5 (Pin_5); no longer J7.6 (Pin_6)
- net at U5.8 (OUT1), U5.9 (OUT1): now also J7.6 (Pin_6); no longer J7.5 (Pin_5)
Changed lines of the file:
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@@
+	)
+	(junction
+		(at 107.95 204.47)
+		(diameter 0)
+		(color 0 0 0 0)
 	)
 	(junction
@@
 	)
 	(junction
-		(at 107.95 207.01)
-		(diameter 0)
-		(color 0 0 0 0)
-	)
-	(junction
 		(at 59.69 130.81)
 		(diameter 0)
@@
 	(wire
 		(pts
-			(xy 111.76 204.47) (xy 111.76 214.63)
+			(xy 111.76 207.01) (xy 111.76 214.63)
 		)
 		(stroke
@@
 	(wire
 		(pts
-			(xy 107.95 207.01) (xy 133.35 207.01)
-		)
-		(stroke
-			(width 0)
-			(type default)
-		)
-	)
-	(wire
-		(pts
 			(xy 229.87 147.32) (xy 245.11 147.32)
 		)
@@
 	(wire
 		(pts
+			(xy 111.76 207.01) (xy 133.35 207.01)
+		)
+		(stroke
+			(width 0)
+			(type default)
+		)
+	)
+	(wire
+		(pts
 			(xy 152.4 290.83) (xy 162.56 290.83)
 		)
@@
 	(wire
 		(pts
-			(xy 111.76 204.47) (xy 133.35 204.47)
+			(xy 111.76 214.63) (xy 111.76 217.17)
 		)
 		(stroke
@@
 	(wire
 		(pts
-			(xy 111.76 217.17) (xy 111.76 214.63)
-		)
-		(stroke
-			(width 0)
-			(type default)
-		)
-	)
-	(wire
-		(pts
 			(xy 35.56 133.35) (xy 25.4 133.35)
 		)
@@
 		)
 		(stroke
+			(width 0)
+			(type default)
+		)
+	)
+	(wire
+		(pts
+			(xy 107.95 204.47) (xy 133.35 204.47)
+		)
+		(stroke

Commit message: vault backup: 2025-04-25 03:02:18
Parts:
- BTSEL1: footprint Button_Switch_THT:SW_PUSH_6mm -> Button_Switch_THT:SW_PUSH_1P1T_6x3.5mm_H5.0_APEM_MJTP1250
Changed lines of the file:
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@@
 			)
 		)
-		(property "Footprint" "Button_Switch_THT:SW_PUSH_6mm"
+		(property "Footprint" "Button_Switch_THT:SW_PUSH_1P1T_6x3.5mm_H5.0_APEM_MJTP1250"
 			(at 27.94 95.25 0)
 			(effects
