File: PCBs/ModuleBoard/RP2040_minimal_r2/SwerveModuleBoard.kicad_sch (KiCad schematic)
At the start: 57 parts, among them IC1 AS5600-ASOT, J1 USB_B_Micro, J3 Conn_02x08_Odd_Even_MountingP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, J4 Conn_01x07, J5 Conn_01x06_Pin, J6 Conn_01x02, J7 Conn_01x06_Pin, J8 Conn_01x06, U2 W25Q128JVS, U3 RP2040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

Commit message: vault backup: 2025-04-25 03:17:35
Parts:
- J4: footprint Connector_PinSocket_2.54mm:PinSocket_1x07_P2.54mm_Vertical -> Connector_PinHeader_2.54mm:PinHeader_2x05_P2.54mm_Vertical; symbol Connector_Generic:Conn_01x07 -> Connector_Generic:Conn_02x05_Counter_Clockwise
Connections:
- net +3V3: now also J4.9 (Pin_9)
- net GND: now also J4.1 (Pin_1), J4.10 (Pin_10)
- net GPIO23: now also J4.8 (Pin_8); no longer J4.1 (Pin_1)

Commit message: vault backup: 2025-04-25 03:37:54
Connections:
- net +3V3: now also J4.3 (Pin_3); no longer J4.9 (Pin_9)
- net GND: now also J4.2 (Pin_2); no longer J4.10 (Pin_10)
- net GPIO23: now also J4.4 (Pin_4); no longer J4.8 (Pin_8)
- net GPIO24: now also J4.6 (Pin_6); no longer J4.2 (Pin_2)
- net GPIO25: now also J4.10 (Pin_10); no longer J4.3 (Pin_3)
- net GPIO26_ADC0: now also J4.8 (Pin_8); no longer J4.4 (Pin_4)
- net GPIO27_ADC1: now also J4.9 (Pin_9); no longer J4.5 (Pin_5)
- net GPIO28_ADC2: now also J4.7 (Pin_7); no longer J4.6 (Pin_6)
- net GPIO29_ADC3: now also J4.5 (Pin_5); no longer J4.7 (Pin_7)
Other:
- moved on the sheet: J4

Commit message: vault backup: 2025-04-25 04:03:28
Parts:
- removed J8: Conn_01x06, Connector_PinHeader_2.54mm:PinHeader_1x06_P2.54mm_Vertical, symbol Connector_Generic:Conn_01x06
- added J2: Conn_02x02_Counter_Clockwise, symbol Connector_Generic:Conn_02x02_Counter_Clockwise
Connections:
- net +3V3: now also J2.2 (Pin_2)
- net GND: now also J2.3 (Pin_3)
- net GPIO0: now also J2.4 (Pin_4)
- net GPIO1: now also J2.1 (Pin_1)
Changed lines of the file:
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@@
 	(wire
 		(pts
+			(xy 267.97 120.65) (xy 283.21 120.65)
+		)
+		(stroke
+			(width 0)
+			(type default)
+		)
+	)
+	(wire
+		(pts
 			(xy 157.48 71.12) (xy 168.91 71.12)
 		)
@@
 	(wire
 		(pts
+			(xy 304.8 120.65) (xy 304.8 121.92)
+		)
+		(stroke
+			(width 0)
+			(type default)
+		)
+	)
+	(wire
+		(pts
 			(xy 360.68 179.07) (xy 360.68 171.45)
 		)
@@
 	(wire
 		(pts
+			(xy 295.91 120.65) (xy 304.8 120.65)
+		)
+		(stroke
+			(width 0)
+			(type default)
+		)
+	)
+	(wire
+		(pts
 			(xy 234.95 222.25) (xy 246.38 222.25)
 		)
@@
 		)
 	)
+	(label "GPIO1"
+		(at 283.21 118.11 180)
+		(effects
+			(font
+				(size 1.27 1.27)
+			)
+			(justify right bottom)
+		)
+	)
 	(label "SCL1"
 		(at 247.65 119.38 0)
@@
 		)
 	)
+	(label "GPIO0"
+		(at 295.91 118.11 0)
+		(effects
+			(font
+				(size 1.27 1.27)
+			)
+			(justify left bottom)
+		)
+	)
 	(label "GPIO15"
 		(at 245.11 149.86 180)
@@
 	)
 	(symbol
+		(lib_name "+3V3_6")
+		(lib_id "power:+3V3")
+		(at 267.97 120.65 0)
+		(unit 1)
+		(exclude_from_sim no)
+		(in_bom yes)
+		(on_board yes)
+		(dnp no)
+		(fields_autoplaced yes)
+		(property "Reference" "#PWR050"
+			(at 267.97 124.46 0)
+			(effects
+				(font
+					(size 1.27 1.27)
+				)
+				(hide yes)
+			)
+		)
+		(property "Value" "+3V3"
+			(at 267.97 115.57 0)
+			(effects
+				(font
+					(size 1.27 1.27)
+				)
+			)
+		)
+		(property "Footprint" ""
+			(at 267.97 120.65 0)
+			(effects
+				(font
+					(size 1.27 1.27)
+				)
+				(hide yes)
+			)
+		)
+		(property "Datasheet" ""
+			(at 267.97 120.65 0)
+			(effects
+				(font
+					(size 1.27 1.27)
+				)
+				(hide yes)
+			)
+		)
+		(property "Description" "Power symbol creates a global label with name \"+3V3\""
+			(at 267.97 120.65 0)
+			(effects
+				(font
+					(size 1.27 1.27)
+				)
+				(hide yes)
+			)
+		)
+		(pin "1"
+		)
+		(instances
+			(project ""
+				(path "/8c0b3d8b-46d3-4173-ab1e-a61765f77d61"
+					(reference "#PWR050")
+					(unit 1)
+				)
+			)
+		)
+	)
+	(symbol
 		(lib_id "2025-04-08_02-58-05:DRV8245HQRXZRQ1")
 		(at 314.96 168.91 0)
@@
 	)
 	(symbol
-		(lib_id "Connector_Generic:Conn_01x06")
-		(at 261.62 116.84 0)
-		(unit 1)
-		(exclude_from_sim no)
-		(in_bom yes)
-		(on_board yes)
-		(dnp no)
-		(fields_autoplaced yes)
-		(property "Reference" "J8"
-			(at 264.16 116.8399 0)
-			(effects
-				(font
-					(size 1.27 1.27)
-				)
-				(justify left)
-			)
-		)
-		(property "Value" "Conn_01x06"
-			(at 264.16 119.3799 0)
-			(effects
-				(font
-					(size 1.27 1.27)
-				)
-				(justify left)
-			)
-		)
-		(property "Footprint" "Connector_PinHeader_2.54mm:PinHeader_1x06_P2.54mm_Vertical"
-			(at 261.62 116.84 0)
-			(effects
-				(font
-					(size 1.27 1.27)
-				)
-				(hide yes)
-			)
-		)
-		(property "Datasheet" "~"
-			(at 261.62 116.84 0)
-			(effects
-				(font
-					(size 1.27 1.27)
-				)
-				(hide yes)
-			)
-		)
-		(property "Description" "Generic connector, single row, 01x06, script generated (kicad-library-utils/schlib/autogen/connector/)"
-			(at 261.62 116.84 0)
-			(effects
-				(font
-					(size 1.27 1.27)
-				)
-				(hide yes)
-			)
-		)
-		(pin "3"
-		)
-		(pin "2"
-		)
-		(pin "4"
-		)
-		(pin "1"
-		)
-		(pin "5"
-		)
-		(pin "6"
-		)
-		(instances
-			(project ""
-				(path "/8c0b3d8b-46d3-4173-ab1e-a61765f77d61"
-					(reference "J8")
-					(unit 1)
-				)
-			)
-		)
-	)
-	(symbol
 		(lib_id "Regulator_Linear:MIC5219-3.3YM5")
 		(at 144.78 293.37 0)
@@
 	)
 	(symbol
+		(lib_name "GND_11")
+		(lib_id "power:GND")
+		(at 304.8 121.92 0)
+		(unit 1)
+		(exclude_from_sim no)
+		(in_bom yes)
+		(on_board yes)
+		(dnp no)
+		(fields_autoplaced yes)
+		(property "Reference" "#PWR049"
+			(at 304.8 128.27 0)
+			(effects
+				(font
+					(size 1.27 1.27)
+				)
+				(hide yes)
+			)
+		)
+		(property "Value" "GND"
+			(at 304.8 127 0)
+			(effects
+				(font
+					(size 1.27 1.27)
+				)
+			)
+		)
+		(property "Footprint" ""
+			(at 304.8 121.92 0)
+			(effects
+				(font
+					(size 1.27 1.27)
+				)
+				(hide yes)
+			)
+		)
+		(property "Datasheet" ""
+			(at 304.8 121.92 0)
+			(effects
+				(font
+					(size 1.27 1.27)
+				)
+				(hide yes)
+			)
+		)
+		(property "Description" "Power symbol creates a global label with name \"GND\" , ground"
+			(at 304.8 121.92 0)
+			(effects
+				(font
+					(size 1.27 1.27)
+				)
+				(hide yes)
+			)
+		)
+		(pin "1"
+		)
+		(instances
+			(project ""
+				(path "/8c0b3d8b-46d3-4173-ab1e-a61765f77d61"
+					(reference "#PWR049")
+					(unit 1)
+				)
+			)
+		)
+	)
+	(symbol
 		(lib_id "Connector:Conn_01x06_Pin")
 		(at 138.43 212.09 180)
@@
 					(unit 1)
 				)
+			)
+		)
+	)
+	(symbol
+		(lib_id "Connector_Generic:Conn_02x02_Counter_Clockwise")
+		(at 288.29 118.11 0)
+		(unit 1)
+		(exclude_from_sim no)
+		(in_bom yes)
+		(on_board yes)
+		(dnp no)
+		(fields_autoplaced yes)
+		(property "Reference" "J2"
+			(at 289.56 111.76 0)
+			(effects
+				(font
+					(size 1.27 1.27)
+				)
+			)
+		)
+		(property "Value" "Conn_02x02_Counter_Clockwise"
+			(at 289.56 114.3 0)
+			(effects
+				(font
+					(size 1.27 1.27)
+				)
+			)
+		)
+		(property "Footprint" ""
+			(at 288.29 118.11 0)
+			(effects
+				(font
+					(size 1.27 1.27)
+				)
+				(hide yes)
+			)
+		)
+		(property "Datasheet" "~"
+			(at 288.29 118.11 0)
+			(effects
+				(font
+					(size 1.27 1.27)
+				)
+				(hide yes)
+			)
+		)
+		(property "Description" "Generic connector, double row, 02x02, counter clockwise pin numbering scheme (similar to DIP package numbering), script generated (kicad-library-utils/schlib/autogen/connector/)"
+			(at 288.29 118.11 0)
+			(effects
+				(font
+					(size 1.27 1.27)
+				)
+				(hide yes)
+			)
+		)
+		(pin "4"
+		)
+		(pin "1"
+		)
+		(pin "3"
+		)
+		(pin "2"
+		)
+		(instances
+			(project ""
+				(path "/8c0b3d8b-46d3-4173-ab1e-a61765f77d61"
+					(reference "J2")
+					(unit 1)
+				)

Commit message: vault backup: 2025-04-25 04:08:35
Parts:
- J2: footprint (none) -> Connector_PinHeader_2.54mm:PinHeader_2x02_P2.54mm_Vertical
Changed lines of the file:
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@@
 			)
 		)
-		(property "Footprint" ""
+		(property "Footprint" "Connector_PinHeader_2.54mm:PinHeader_2x02_P2.54mm_Vertical"
 			(at 288.29 118.11 0)
 			(effects

Commit message: vault backup: 2025-04-25 04:13:42
Connections:
- net GND: now also J2.1 (Pin_1); no longer J2.3 (Pin_3)
- net GPIO1: now also J2.3 (Pin_3); no longer J2.1 (Pin_1)
Changed lines of the file:
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@@
 	(wire
 		(pts
-			(xy 304.8 120.65) (xy 304.8 121.92)
+			(xy 360.68 179.07) (xy 360.68 171.45)
 		)
 		(stroke
@@
 	(wire
 		(pts
-			(xy 360.68 179.07) (xy 360.68 171.45)
+			(xy 53.34 184.15) (xy 53.34 186.69)
 		)
 		(stroke
@@
 	(wire
 		(pts
-			(xy 53.34 184.15) (xy 53.34 186.69)
+			(xy 276.86 116.84) (xy 283.21 116.84)
 		)
 		(stroke
@@
 	(wire
 		(pts
-			(xy 295.91 120.65) (xy 304.8 120.65)
-		)
-		(stroke
-			(width 0)
-			(type default)
-		)
-	)
-	(wire
-		(pts
 			(xy 234.95 222.25) (xy 246.38 222.25)
 		)
@@
 	(wire
 		(pts
+			(xy 283.21 116.84) (xy 283.21 118.11)
+		)
+		(stroke
+			(width 0)
+			(type default)
+		)
+	)
+	(wire
+		(pts
 			(xy 280.67 60.96) (xy 292.1 60.96)
 		)
@@
 		)
 	)
-	(label "GPIO1"
-		(at 283.21 118.11 180)
-		(effects
-			(font
-				(size 1.27 1.27)
-			)
-			(justify right bottom)
-		)
-	)
 	(label "SCL1"
 		(at 247.65 119.38 0)
@@
 		)
 	)
+	(label "GPIO1"
+		(at 295.91 120.65 0)
+		(effects
+			(font
+				(size 1.27 1.27)
+			)
+			(justify left bottom)
+		)
+	)
 	(label "QSPI_SD0"
 		(at 73.66 105.41 0)
@@
 		(lib_name "GND_11")
 		(lib_id "power:GND")
-		(at 304.8 121.92 0)
+		(at 276.86 116.84 0)
 		(unit 1)
 		(exclude_from_sim no)
@@
 		(fields_autoplaced yes)
 		(property "Reference" "#PWR049"
-			(at 304.8 128.27 0)
+			(at 276.86 123.19 0)
 			(effects
 				(font
@@
 		)
 		(property "Value" "GND"
-			(at 304.8 127 0)
+			(at 276.86 121.92 0)
 			(effects
 				(font
@@
 		)
 		(property "Footprint" ""
-			(at 304.8 121.92 0)
+			(at 276.86 116.84 0)
 			(effects
 				(font
@@
 		)
 		(property "Datasheet" ""
-			(at 304.8 121.92 0)
+			(at 276.86 116.84 0)
 			(effects
 				(font
@@
 		)
 		(property "Description" "Power symbol creates a global label with name \"GND\" , ground"
-			(at 304.8 121.92 0)
+			(at 276.86 116.84 0)
 			(effects
 				(font

Commit message: vault backup: 2025-04-25 05:55:47
Parts:
- added D4, D7, D8, D9: WS2812B, LED_SMD:LED_WS2812B_PLCC4_5.0x5.0mm_P3.2mm, symbol LED:WS2812B
Connections:
- net +5V: now also D4.1 (VDD), D7.1 (VDD), D8.1 (VDD), D9.1 (VDD)
- net GND: now also D4.3 (VSS), D7.3 (VSS), D8.3 (VSS), D9.3 (VSS)
- net GPIO23: now also D4.4 (DIN)
- new net: D7.2 (DOUT), D8.4 (DIN)
- new net: D4.2 (DOUT), D7.4 (DIN)
- new net: D8.2 (DOUT), D9.4 (DIN)
- no-connect marks 5 -> 6

Commit message: vault backup: 2025-04-25 06:06:02
Connections:
- net +5V: now also J3.13 (Pin_13)
- no-connect marks 6 -> 5
Changed lines of the file:
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@@
+	)
+	(junction
+		(at 54.61 151.13)
+		(diameter 0)
+		(color 0 0 0 0)
 	)
 	(junction
@@
 	)
 	(no_connect
-		(at 34.29 146.05)
-	)
-	(no_connect
 		(at 41.91 153.67)
 	)
@@
 	(wire
 		(pts
+			(xy 29.21 146.05) (xy 29.21 163.83)
+		)
+		(stroke
+			(width 0)
+			(type default)
+		)
+	)
+	(wire
+		(pts
 			(xy 87.63 142.24) (xy 87.63 143.51)
 		)
@@
 	(wire
 		(pts
+			(xy 29.21 163.83) (xy 54.61 163.83)
+		)
+		(stroke
+			(width 0)
+			(type default)
+		)
+	)
+	(wire
+		(pts
 			(xy 152.4 290.83) (xy 162.56 290.83)
 		)
@@
 	(wire
 		(pts
-			(xy 34.29 146.05) (xy 35.56 146.05)
-		)
-		(stroke
-			(width 0)
-			(type default)
-		)
-	)
-	(wire
-		(pts
 			(xy 144.78 302.26) (xy 144.78 300.99)
 		)
@@
 	(wire
 		(pts
+			(xy 29.21 146.05) (xy 35.56 146.05)
+		)
+		(stroke
+			(width 0)
+			(type default)
+		)
+	)
+	(wire
+		(pts
 			(xy 228.6 228.6) (xy 238.76 228.6)
 		)
@@
 		)
 		(stroke
+			(width 0)
+			(type default)
+		)
+	)
+	(wire
+		(pts
+			(xy 54.61 163.83) (xy 54.61 151.13)
+		)
+		(stroke

Commit message: vault backup: 2025-04-25 21:40:27
Parts:
- added R12: 470, Capacitor_SMD:C_0603_1608Metric_Pad1.08x0.95mm_HandSolder, symbol Device:R
Connections:
- net GPIO23: now also R12.1; no longer D4.4 (DIN), J4.4 (Pin_4)
- new net GPIO23R: D4.4 (DIN), J4.4 (Pin_4), R12.2
Changed lines of the file:
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@@
 	)
 	(junction
-		(at 234.95 222.25)
-		(diameter 0)
-		(color 0 0 0 0)
-	)
-	(junction
 		(at 280.67 60.96)
 		(diameter 0)
@@
 	)
 	(junction
+		(at 234.95 219.71)
+		(diameter 0)
+		(color 0 0 0 0)
+	)
+	(junction
 		(at 22.86 140.97)
 		(diameter 0)
@@
 	(wire
 		(pts
+			(xy 234.95 210.82) (xy 234.95 219.71)
+		)
+		(stroke
+			(width 0)
+			(type default)
+		)
+	)
+	(wire
+		(pts
 			(xy 207.01 81.28) (xy 210.82 81.28)
 		)
@@
 	(wire
 		(pts
+			(xy 358.14 267.97) (xy 358.14 264.16)
+		)
+		(stroke
+			(width 0)
+			(type default)
+		)
+	)
+	(wire
+		(pts
 			(xy 318.77 80.01) (xy 322.58 80.01)
 		)
@@
 	(wire
 		(pts
+			(xy 355.6 267.97) (xy 358.14 267.97)
+		)
+		(stroke
+			(width 0)
+			(type default)
+		)
+	)
+	(wire
+		(pts
 			(xy 248.92 96.52) (xy 262.89 96.52)
 		)
@@
 	(wire
 		(pts
-			(xy 81.28 295.91) (xy 90.17 295.91)
+			(xy 358.14 264.16) (xy 363.22 264.16)
 		)
 		(stroke
@@
 	(wire
 		(pts
-			(xy 177.8 60.96) (xy 177.8 76.2)
+			(xy 81.28 295.91) (xy 90.17 295.91)
 		)
 		(stroke
@@
 	(wire
 		(pts
-			(xy 295.91 151.13) (xy 302.26 151.13)
+			(xy 177.8 60.96) (xy 177.8 76.2)
 		)
 		(stroke
@@
 	(wire
 		(pts
-			(xy 210.82 81.28) (xy 214.63 81.28)
+			(xy 295.91 151.13) (xy 302.26 151.13)
 		)
 		(stroke
@@
 	(wire
 		(pts
-			(xy 152.4 119.38) (xy 166.37 119.38)
+			(xy 210.82 81.28) (xy 214.63 81.28)
 		)
 		(stroke
@@
 	(wire
 		(pts
-			(xy 228.6 228.6) (xy 228.6 224.79)
+			(xy 152.4 119.38) (xy 166.37 119.38)
 		)
 		(stroke
@@
 	(wire
 		(pts
-			(xy 238.76 224.79) (xy 246.38 224.79)
-		)
-		(stroke
-			(width 0)
-			(type default)
-		)
-	)
-	(wire
-		(pts
 			(xy 111.76 207.01) (xy 111.76 214.63)
 		)
@@
 	(wire
 		(pts
+			(xy 228.6 210.82) (xy 234.95 210.82)
+		)
+		(stroke
+			(width 0)
+			(type default)
+		)
+	)
+	(wire
+		(pts
 			(xy 25.4 130.81) (xy 25.4 133.35)
 		)
@@
 	(wire
 		(pts
+			(xy 346.71 264.16) (xy 339.09 264.16)
+		)
+		(stroke
+			(width 0)
+			(type default)
+		)
+	)
+	(wire
+		(pts
 			(xy 360.68 171.45) (xy 382.27 171.45)
 		)
@@
 	(wire
 		(pts
+			(xy 346.71 267.97) (xy 346.71 264.16)
+		)
+		(stroke
+			(width 0)
+			(type default)
+		)
+	)
+	(wire
+		(pts
 			(xy 46.99 191.77) (xy 46.99 186.69)
 		)
@@
 	(wire
 		(pts
-			(xy 228.6 228.6) (xy 238.76 228.6)
+			(xy 228.6 224.79) (xy 246.38 224.79)
 		)
 		(stroke
@@
 	(wire
 		(pts
+			(xy 346.71 267.97) (xy 347.98 267.97)
+		)
+		(stroke
+			(width 0)
+			(type default)
+		)
+	)
+	(wire
+		(pts
 			(xy 257.81 69.85) (xy 257.81 72.39)
 		)
@@
 	(wire
 		(pts
-			(xy 238.76 228.6) (xy 238.76 224.79)
+			(xy 234.95 219.71) (xy 234.95 222.25)
 		)
 		(stroke
@@
 	(wire
 		(pts
-			(xy 234.95 219.71) (xy 234.95 222.25)
-		)
-		(stroke
-			(width 0)
-			(type default)
-		)
-	)
-	(wire
-		(pts
 			(xy 71.12 307.34) (xy 71.12 308.61)
 		)
@@
 		)
 	)
+	(label "GPIO23"
+		(at 339.09 264.16 180)
+		(effects
+			(font
+				(size 1.27 1.27)
+			)
+			(justify right bottom)
+		)
+	)
 	(label "QSPI_SS"
 		(at 73.66 100.33 0)
@@
 		)
 	)
-	(label "GPIO23"
-		(at 363.22 264.16 180)
-		(effects
-			(font
-				(size 1.27 1.27)
-			)
-			(justify right bottom)
-		)
-	)
 	(label "GPIO21"
 		(at 245.11 165.1 180)
@@
 		)
 	)
-	(label "GPIO23"
-		(at 246.38 227.33 180)
-		(effects
-			(font
-				(size 1.27 1.27)
-			)
-			(justify right bottom)
-		)
-	)
 	(label "GPIO9"
 		(at 245.11 134.62 180)
@@
 		)
 	)
+	(global_label "GPIO23R"
+		(shape input)
+		(at 358.14 264.16 90)
+		(fields_autoplaced yes)
+		(effects
+			(font
+				(size 1.27 1.27)
+			)
+			(justify left)
+		)
+		(property "Intersheetrefs" "${INTERSHEET_REFS}"
+			(at 358.14 253.6647 90)
+			(effects
+				(font
+					(size 1.27 1.27)
+				)
+				(justify left)
+				(hide yes)
+			)
+		)
+	)
+	(global_label "GPIO23R"
+		(shape input)
+		(at 246.38 227.33 180)
+		(fields_autoplaced yes)
+		(effects
+			(font
+				(size 1.27 1.27)
+			)
+			(justify right)
+		)
+		(property "Intersheetrefs" "${INTERSHEET_REFS}"
+			(at 235.8847 227.33 0)
+			(effects
+				(font
+					(size 1.27 1.27)
+				)
+				(justify right)
+				(hide yes)
+			)
+		)
+	)
 	(symbol
 		(lib_id "MCU_RaspberryPi_RP2040:RP2040")
@@
 		(lib_name "GND_10")
 		(lib_id "power:GND")
-		(at 234.95 222.25 0)
+		(at 228.6 210.82 0)
 		(unit 1)
 		(exclude_from_sim no)
@@
 		(fields_autoplaced yes)
 		(property "Reference" "#PWR09"
-			(at 234.95 228.6 0)
+			(at 228.6 217.17 0)
 			(effects
 				(font
@@
 		)
 		(property "Value" "GND"
-			(at 234.95 227.33 0)
+			(at 228.6 215.9 0)
 			(effects
 				(font
@@
 		)
 		(property "Footprint" ""
-			(at 234.95 222.25 0)
+			(at 228.6 210.82 0)
 			(effects
 				(font
@@
 		)
 		(property "Datasheet" ""
-			(at 234.95 222.25 0)
+			(at 228.6 210.82 0)
 			(effects
 				(font
@@
 		)
 		(property "Description" "Power symbol creates a global label with name \"GND\" , ground"
-			(at 234.95 222.25 0)
+			(at 228.6 210.82 0)
 			(effects
 				(font
@@
 					(unit 1)
 				)
+			)
+		)
+	)
+	(symbol
+		(lib_id "Device:R")
+		(at 351.79 267.97 90)
+		(unit 1)
+		(exclude_from_sim no)
+		(in_bom yes)
+		(on_board yes)
+		(dnp no)
+		(fields_autoplaced yes)
+		(property "Reference" "R12"
+			(at 351.79 261.62 90)
+			(effects
+				(font
+					(size 1.27 1.27)
+				)
+			)
+		)
+		(property "Value" "470"
+			(at 351.79 264.16 90)
+			(effects
+				(font
+					(size 1.27 1.27)
+				)
+			)
+		)
+		(property "Footprint" "Capacitor_SMD:C_0603_1608Metric_Pad1.08x0.95mm_HandSolder"
+			(at 351.79 269.748 90)
+			(effects
+				(font
+					(size 1.27 1.27)
+				)
+				(hide yes)
+			)
+		)
+		(property "Datasheet" "~"
+			(at 351.79 267.97 0)
+			(effects
+				(font
+					(size 1.27 1.27)
+				)
+				(hide yes)
+			)
+		)
+		(property "Description" "Resistor"
+			(at 351.79 267.97 0)
+			(effects
+				(font
+					(size 1.27 1.27)
+				)
+				(hide yes)
+			)
+		)
+		(pin "1"
+		)
+		(pin "2"
+		)
+		(instances
+			(project ""
+				(path "/8c0b3d8b-46d3-4173-ab1e-a61765f77d61"
+					(reference "R12")
+					(unit 1)
+				)
