File: PCBs/ModuleBoard/RP2040_minimal_r2/SwerveModuleBoard.kicad_pcb (KiCad board)
At the start: 2 copper layers, 60 x 52.9 mm, 54 parts, among them IC1 AS5600-ASOT, J1 USB_B_Micro, J3 Conn_02x08_Odd_Even_MountingP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, J4 Conn_01x07, J5 Conn_01x06_Pin, J6 Conn_01x02, J7 Conn_01x06_Pin, J8 Conn_01x06, U1 NCP1117-3.3_SOT223, U2 W25Q128JVS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

Commit message: vault backup: 2025-04-25 01:51:37
Parts:
- removed C1, C4: 10u, Capacitor_SMD:C_0603_1608Metric_Pad1.08x0.95mm_HandSolder
- removed U1: NCP1117-3.3_SOT223, Package_TO_SOT_SMD:SOT-223-3_TabPin2
- added C25: 10μF, Capacitor_SMD:C_0603_1608Metric_Pad1.08x0.95mm_HandSolder, F.Cu at (111.8, 80.0)
- added C26: 1nF, Capacitor_SMD:C_0603_1608Metric_Pad1.08x0.95mm_HandSolder, F.Cu at (104.2, 81.5)
- added C27: 10μF, Capacitor_SMD:C_0603_1608Metric_Pad1.08x0.95mm_HandSolder, F.Cu at (104.2, 79.8)
- added D3: 1n4007, Diode_SMD:D_SOD-123, F.Cu at (106.2, 74.0)
- added D4: 1n4007, Diode_SMD:D_SOD-123, F.Cu at (124.0, 111.5)
- added L2: 1.5 μH, Capacitor_SMD:C_0603_1608Metric_Pad1.08x0.95mm_HandSolder, F.Cu at (110.8, 77.5)
- added R12: 1M, Resistor_SMD:R_0603_1608Metric_Pad0.98x0.95mm_HandSolder, F.Cu at (107.8, 83.2)
- added U7: TPS63051RMWR, BuckBoost:QFN50P250X250X100-12N, F.Cu at (108.8, 80.2)
- U2: footprint Package_SO:SOIC-8_5.23x5.23mm_P1.27mm -> Package_SO:SOIC-8_5.3x5.3mm_P1.27mm
- moved J7 42.3 mm to (125.0, 105.8), turned to 180 degrees
- moved U5 42.3 mm to (119.7, 97.8), turned to 90 degrees
- moved J4 24.8 mm to (136.0, 83.6)
- moved J6 5.51 mm to (116.2, 113.8), turned to -90 degrees
- moved R11 5.31 mm to (107.0, 95.8), turned to 0 degrees
- moved D2 1.11 mm to (106.9, 94.0)
Routing:
- net Net-(D3-K): track 0.00 -> 58.2 mm
- net GND: track 109.2 -> 121.8 mm, vias 46 -> 51
- net +3V3: track 109.2 -> 103.9 mm, vias 3 -> 2
- net Net-(U7-SS): track 0.00 -> 2.93 mm
- net Net-(U7-L1): track 0.00 -> 2.73 mm
- net Net-(U7-L2): track 0.00 -> 2.39 mm
- net VBUS: track 8.55 -> 6.23 mm
- net Net-(U7-PG): track 0.00 -> 1.88 mm
- net /GPIO22: track 7.10 -> 6.39 mm

Commit message: vault backup: 2025-04-25 03:02:18
Parts:
- removed C25, C27: 10μF, Capacitor_SMD:C_0603_1608Metric_Pad1.08x0.95mm_HandSolder
- removed C26: 1nF, Capacitor_SMD:C_0603_1608Metric_Pad1.08x0.95mm_HandSolder
- removed D3, D4: 1n4007, Diode_SMD:D_SOD-123
- removed L2: 1.5 μH, Capacitor_SMD:C_0603_1608Metric_Pad1.08x0.95mm_HandSolder
- removed R12: 1M, Resistor_SMD:R_0603_1608Metric_Pad0.98x0.95mm_HandSolder
- removed U7: TPS63051RMWR, BuckBoost:QFN50P250X250X100-12N
- added C23: 470 pF, Capacitor_SMD:C_0603_1608Metric, F.Cu at (105.8, 83.8)
- added C24: 22 uF, Capacitor_SMD:C_1206_3216Metric_Pad1.33x1.80mm_HandSolder, F.Cu at (111.0, 75.0)
- added D5: PMEG3020EXEX, Diode_SMD:D_SOD-123F, F.Cu at (110.5, 81.2)
- added D6: PMEG3020EXEX, Diode_SMD:D_SOD-123F, F.Cu at (102.8, 78.2)
- added R13: 10k, Resistor_SMD:R_0603_1608Metric, F.Cu at (102.5, 81.8)
- added U6: MIC5219-3.3YM5, Package_TO_SOT_SMD:SOT-23-5, F.Cu at (106.2, 81.0)
- moved J5 54.9 mm to (75.0, 93.2), turned to 0 degrees
- moved C18 49.0 mm to (119.8, 88.8)
- moved R9 37.5 mm to (114.5, 96.5), turned to 90 degrees
- moved U4 35.5 mm to (80.8, 104.8), turned to -90 degrees
- moved C21 34.6 mm to (120.2, 107.8)
- moved C22 31.9 mm to (104.5, 96.8)
- moved J8 20.8 mm to (60.0, 71.4)
- moved J4 8.05 mm to (143.3, 80.2), turned to -90 degrees
- moved U5 3.29 mm to (119.5, 94.5)
- moved R8 2.85 mm to (103.8, 101.5)
- moved R10 2.15 mm to (108.8, 99.2)
- moved D1 0.52 mm to (106.9, 97.5)
Connections:
- J3 pad 14: unconnected-(J3-Pin_14-Pad14) -> +5V
- U5 pad 5: Net-(J7-Pin_6) -> Net-(J7-Pin_5)
- U5 pad 6: Net-(J7-Pin_6) -> Net-(J7-Pin_5)
- U5 pad 8: Net-(J7-Pin_5) -> Net-(J7-Pin_6)
- U5 pad 9: Net-(J7-Pin_5) -> Net-(J7-Pin_6)
Routing:
- net +5V: track 0.00 -> 84.4 mm
- net +3V3: track 103.9 -> 168.2 mm, vias 2 -> 4
- net Net-(D3-K): track 58.2 -> 0.00 mm
- net VM: track 51.4 -> 103.5 mm
- net /GPIO16: track 0.00 -> 25.2 mm
- net /GPIO19: track 0.00 -> 24.2 mm
- net /GPIO20: track 0.00 -> 24.1 mm
- net /GPIO18: track 0.00 -> 23.2 mm
- net /GPIO8: track 0.00 -> 19.1 mm
- net /GPIO9: track 0.00 -> 18.4 mm
- net Net-(J7-Pin_5): track 27.5 -> 11.5 mm
- net /GPIO3: track 0.00 -> 13.8 mm, vias 0 -> 1
- net /GPIO2: track 0.00 -> 12.9 mm, vias 0 -> 1
- net Net-(J5-Pin_5): track 13.2 -> 25.3 mm
- net Net-(J5-Pin_6): track 19.1 -> 31.1 mm
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- added copper zone on B.Cu, net GND

Commit message: vault backup: 2025-04-25 03:12:28
Parts:
- BTSEL1: footprint Button_Switch_THT:SW_PUSH_6mm -> Button_Switch_THT:SW_PUSH_1P1T_6x3.5mm_H5.0_APEM_MJTP1250
- moved R7 38.2 mm to (90.0, 97.2), turned to 180 degrees
- moved C20 29.9 mm to (83.8, 108.5), turned to 180 degrees
- moved R6 27.8 mm to (86.2, 104.8), turned to 180 degrees
- moved C19 26.6 mm to (84.8, 116.8), turned to -90 degrees
- moved J8 6.49 mm to (56.5, 76.8)
- moved BTSEL1 5.52 mm to (82.2, 87.2), turned to 90 degrees
Routing:
- net /GPIO4: track 0.00 -> 63.8 mm
- net /GPIO5: track 0.00 -> 63.6 mm
- net VM: track 103.5 -> 66.6 mm
- net GND: track 125.0 -> 94.7 mm, vias 54 -> 48
- net /GPIO15: track 0.00 -> 19.3 mm
- net Net-(J5-Pin_6): track 31.1 -> 12.1 mm
- net /GPIO14: track 0.00 -> 18.4 mm
- net /GPIO13: track 0.00 -> 16.8 mm
- net /GPIO10: track 0.00 -> 14.9 mm
- net /GPIO12: track 3.83 -> 17.1 mm
- net Net-(J5-Pin_5): track 25.3 -> 12.1 mm
- net +3V3: track 168.2 -> 157.0 mm
- net /~{USB_BOOT}: track 21.9 -> 11.9 mm
- net Net-(U4-SR): track 4.57 -> 2.07 mm

Commit message: vault backup: 2025-04-25 03:43:01
Parts:
- J4: footprint Connector_PinSocket_2.54mm:PinSocket_1x07_P2.54mm_Vertical -> Connector_PinHeader_2.54mm:PinHeader_2x05_P2.54mm_Vertical
- moved J4 27.1 mm to (116.4, 83.5), turned to -45 degrees
- moved BTSEL1 5.61 mm to (76.7, 86.3), turned to 45 degrees
- moved C15 0.66 mm to (107.0, 86.9)
Connections:
- J4 pad 1: /GPIO23 -> GND
- J4 pad 2: /GPIO24 -> GND
- J4 pad 3: /GPIO25 -> +3V3
- J4 pad 4: /GPIO26_ADC0 -> /GPIO23
- J4 pad 5: /GPIO27_ADC1 -> /GPIO29_ADC3
- J4 pad 6: /GPIO28_ADC2 -> /GPIO24
- J4 pad 7: /GPIO29_ADC3 -> /GPIO28_ADC2
Routing:
- net /GPIO23: track 0.00 -> 20.9 mm
- net /GPIO24: track 0.00 -> 18.1 mm
- net /GPIO29_ADC3: track 0.00 -> 14.8 mm
- net /GPIO26_ADC0: track 0.00 -> 13.6 mm
- net /GPIO28_ADC2: track 0.00 -> 12.4 mm
- net /GPIO25: track 0.00 -> 11.2 mm
- net /GPIO27_ADC1: track 0.00 -> 10.2 mm
- net +3V3: track 157.0 -> 165.0 mm
- net /~{USB_BOOT}: track 11.9 -> 13.3 mm

Commit message: vault backup: 2025-04-25 04:34:04
Parts:
- removed J8: Conn_01x06, Connector_PinHeader_2.54mm:PinHeader_1x06_P2.54mm_Vertical
- added J2: Conn_02x02_Counter_Clockwise, Connector_PinHeader_2.54mm:PinHeader_2x02_P2.54mm_Vertical, F.Cu at (81.2, 87.5)
- moved C13 3.28 mm to (86.8, 94.8)
Routing:
- net /GPIO6: track 0.00 -> 42.7 mm, vias 0 -> 2
- net /GPIO7: track 0.00 -> 40.0 mm, vias 0 -> 2
- net +3V3: track 165.0 -> 182.9 mm
- net /GPIO1: track 0.00 -> 11.0 mm
- net /GPIO0: track 0.00 -> 9.74 mm
- net VBUS: track 6.00 -> 3.09 mm
- net /GPIO3: track 13.8 -> 15.8 mm
- net /GPIO2: track 12.9 -> 14.8 mm
- net GND: track 94.7 -> 96.5 mm, vias 48 -> 50
- net /XIN: track 10.7 -> 12.0 mm
- net /GPIO5: track 63.6 -> 63.1 mm
- removed copper zone on F.Cu, net VBUS
