File: PCBs/ModuleBoard/RP2040_minimal_r2/SwerveModuleBoard.kicad_pcb (KiCad board)
At the start: 2 copper layers, 60 x 52.9 mm, 57 parts, among them IC1 AS5600-ASOT, J1 USB_B_Micro, J2 Conn_02x02_Counter_Clockwise, J3 Conn_02x08_Odd_Even_MountingP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, J4 Conn_01x07, J5 Conn_01x06_Pin, J6 Conn_01x02, J7 Conn_01x06_Pin, U2 W25Q128JVS, U3 RP2040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

Commit message: vault backup: 2025-04-25 05:19:58
Other:
- board text removed: "GND"
Changed lines of the file:
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@@
 		(tags "capacitor handsolder")
 		(property "Reference" "C5"
-			(at -2.645 -0.02 180)
+			(at -2.645 -0.695 0)
 			(layer "F.SilkS")
 			(effects
@@
 		(tags "resistor handsolder")
 		(property "Reference" "R2"
-			(at -2.555 -1.51 270)
+			(at -0.25 1.5 270)
 			(layer "F.SilkS")
 			(effects
@@
 		(tags "resistor handsolder")
 		(property "Reference" "R1"
-			(at 2.615 -1.38 90)
+			(at 2.25 0.5 180)
 			(layer "F.SilkS")
 			(effects
@@
 		(tags "capacitor handsolder")
 		(property "Reference" "C17"
-			(at -3.26 0.04 0)
+			(at -0.8 1.475 0)
 			(layer "F.SilkS")
 			(effects
@@
 		)
 	)
-	(gr_text "GND"
-		(at 91.08 71.29 0)
-		(layer "F.SilkS")
-		(effects
-			(font
-				(size 1 1)
-				(thickness 0.15)
-			)
-		)
-	)
 	(gr_text "3V3"
 		(at 81.585 74 0)
@@
 		(min_thickness 0.15)
 		(filled_areas_thickness no)
-		(fill yes
+		(fill
 			(thermal_gap 0.508)
 			(thermal_bridge_width 0.508)
@@
 		(min_thickness 0.15)
 		(filled_areas_thickness no)
-		(fill yes
+		(fill
 			(thermal_gap 0.508)
 			(thermal_bridge_width 0.508)
@@
 		(min_thickness 0.25)
 		(filled_areas_thickness no)
-		(fill yes
+		(fill
 			(thermal_gap 0.5)
 			(thermal_bridge_width 0.5)
@@
 		(min_thickness 0.25)
 		(filled_areas_thickness no)
-		(fill yes
+		(fill
 			(thermal_gap 0.5)
 			(thermal_bridge_width 0.5)
@@
 		(min_thickness 0.2)
 		(filled_areas_thickness no)
-		(fill yes
+		(fill
 			(thermal_gap 0.3)
 			(thermal_bridge_width 0.3)
@@
 		(min_thickness 0.25)
 		(filled_areas_thickness no)
-		(fill yes
+		(fill
 			(thermal_gap 0.5)
 			(thermal_bridge_width 0.5)

Commit message: vault backup: 2025-04-25 05:25:04
Other:
- board text removed: "3V3"
Changed lines of the file:
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@@
 		(tags "capacitor handsolder")
 		(property "Reference" "C10"
-			(at 2.5 0.75 180)
+			(at -2.5 0 0)
 			(layer "F.SilkS")
 			(effects
@@
 		(tags "capacitor handsolder")
 		(property "Reference" "C8"
-			(at 3.25 -0.25 90)
+			(at 2.5 0 180)
 			(layer "F.SilkS")
 			(effects
@@
 		(tags "capacitor handsolder")
 		(property "Reference" "C13"
-			(at 0.025 -1.53 180)
+			(at 0 1.5 180)
 			(layer "F.SilkS")
 			(effects
@@
 		(tags "capacitor handsolder")
 		(property "Reference" "C5"
-			(at -2.645 -0.695 0)
+			(at -2.365 -0.195 90)
 			(layer "F.SilkS")
 			(effects
@@
 		(tags "SOIC SO P-SOP SOP SOP-8 SO SO-8 8S2 S2AE/F K04-056 CASE-751BE SO8W 8-Pin-SOIC PSA W8-2 W8-4 W8MS-1")
 		(property "Reference" "U2"
-			(at 0 -3.6 0)
+			(at -5.25 -1 270)
 			(layer "F.SilkS")
 			(effects
@@
 		(tags "capacitor handsolder")
 		(property "Reference" "C9"
-			(at 2.75 0.25 90)
+			(at 2.25 0 180)
 			(layer "F.SilkS")
 			(effects
@@
 		(tags "capacitor handsolder")
 		(property "Reference" "C14"
-			(at -0.01 -5.07 270)
+			(at 0.1 3.44 270)
 			(layer "F.SilkS")
 			(effects
@@
 		(tags "resistor handsolder")
 		(property "Reference" "R3"
-			(at -2.72 -0.06 270)
+			(at 2.5 0 0)
 			(layer "F.SilkS")
 			(effects
@@
 		(tags "capacitor handsolder")
 		(property "Reference" "C7"
-			(at 0.16 -4.69 270)
+			(at 0.37 -1.71 270)
 			(layer "F.SilkS")
 			(effects
@@
 		(tags "capacitor handsolder")
 		(property "Reference" "C16"
-			(at 0.06 3.91 90)
+			(at 0.21 -1.23 90)
 			(layer "F.SilkS")
 			(effects
@@
 		(tags "QFN DFN_QFN")
 		(property "Reference" "U3"
-			(at -3.71 -4.6 0)
+			(at -4.75 0 90)
 			(layer "F.SilkS")
 			(effects
@@
 		(tags "resistor handsolder")
 		(property "Reference" "R4"
-			(at -2.79 -0.09 270)
+			(at -2.5 0 0)
 			(layer "F.SilkS")
 			(effects
@@
 		(tags "capacitor handsolder")
 		(property "Reference" "C6"
-			(at 0.5 -1.75 180)
+			(at -2.5 -0.5 180)
 			(layer "F.SilkS")
 			(effects
@@
 		(tags "capacitor handsolder")
 		(property "Reference" "C15"
-			(at 0.01 3.47 90)
+			(at 0.01 1.5 90)
 			(layer "F.SilkS")
 			(effects
@@
 		(tags "capacitor")
 		(property "Reference" "C23"
-			(at 0 -1.43 0)
+			(at -3 0 0)
 			(layer "F.SilkS")
 			(effects
@@
 		(tags "PHAP3362A 6mm tact sw THT")
 		(property "Reference" "BTSEL1"
-			(at 3.42 -2.7 45)
+			(at 4.814544 -2.651651 45)
 			(layer "F.SilkS")
 			(effects
@@
 		(tags "capacitor handsolder")
 		(property "Reference" "C24"
-			(at 0 -1.85 0)
+			(at 0 2.25 0)
 			(layer "F.SilkS")
 			(effects
@@
 		(tags "LED handsolder")
 		(property "Reference" "D1"
-			(at 0 -1.43 0)
+			(at -2.875 0 0)
 			(layer "F.SilkS")
 			(effects
@@
 		(tags "capacitor electrolytic")
 		(property "Reference" "C19"
-			(at 0 -3.7 90)
+			(at 0 3.75 90)
 			(layer "F.SilkS")
 			(effects
@@
 		(tags "capacitor handsolder")
 		(property "Reference" "C3"
-			(at 3.22 0.12 0)
+			(at 2.7 0 0)
 			(layer "F.SilkS")
 			(effects
@@
 		(tags "Through hole pin header THT 2x02 2.54mm double row")
 		(property "Reference" "J2"
-			(at 1.27 -2.380001 45)
+			(at -0.846321 5.164087 45)
 			(layer "F.SilkS")
 			(effects
@@
 		(tags "capacitor electrolytic")
 		(property "Reference" "C21"
-			(at 0 -3.7 90)
+			(at 3.75 -2.5 180)
 			(layer "F.SilkS")
 			(effects
@@
 		(tags "resistor handsolder")
 		(property "Reference" "R10"
-			(at 0 -1.43 0)
+			(at 0 -1.5 0)
 			(layer "F.SilkS")
 			(effects
@@
 		(tags "capacitor handsolder")
 		(property "Reference" "C20"
-			(at 0.005 1.395 0)
+			(at 0.005 -1.5 0)
 			(layer "F.SilkS")
 			(effects
@@
 		(tags "resistor handsolder")
 		(property "Reference" "R6"
-			(at 0 -1.43 0)
+			(at 0 1.5 0)
 			(layer "F.SilkS")
 			(effects
@@
 		(tags "resistor handsolder")
 		(property "Reference" "R11"
-			(at 0 -1.43 0)
+			(at 3.25 0 0)
 			(layer "F.SilkS")
 			(effects
@@
 		(tags "Through hole pin header THT 1x06 2.54mm single row")
 		(property "Reference" "J7"
-			(at 0 -2.33 0)
+			(at -0.25 -2.67 0)
 			(layer "F.SilkS")
 			(effects
@@
 		(tags "RC Connector XT30")
 		(property "Reference" "J6"
-			(at 2.5 -4 90)
+			(at 0 4 90)
 			(layer "F.SilkS")
 			(effects
@@
 		)
 		(fp_text user "+"
-			(at 9 0 90)
+			(at 5.25 -3.75 90)
 			(layer "F.SilkS")
 			(effects
@@
 		)
 		(fp_text user "-"
-			(at -4 0 90)
+			(at 0 -3.5 90)
 			(layer "F.SilkS")
 			(effects
@@
 		(tags "capacitor")
 		(property "Reference" "C22"
-			(at 0 -1.43 90)
+			(at 0.25 1.5 270)
 			(layer "F.SilkS")
 			(effects
@@
 		(tags "resistor handsolder")
 		(property "Reference" "R5"
-			(at -0.08 -5.2 270)
+			(at 0.19 3.08 90)
 			(layer "F.SilkS")
 			(effects
@@
 		(tags "DRV8245HQRXZRQ1 ")
 		(property "Reference" "U5"
-			(at 0 0 90)
+			(at -3.037501 0.394857 0)
 			(unlocked yes)
 			(layer "F.SilkS")
@@
 		)
 		(fp_text user "DRV8245"
-			(at 7.915 -0.905 90)
+			(at 2.962499 -0.249999 0)
 			(unlocked yes)
 			(layer "F.SilkS")
@@
 		(tags "resistor handsolder")
 		(property "Reference" "R8"
-			(at 0 -1.43 0)
+			(at 0 1.5 0)
 			(layer "F.SilkS")
 			(effects
@@
 		(tags "DRV8245HQRXZRQ1 ")
 		(property "Reference" "U4"
-			(at -4.777499 0.435001 270)
+			(at 3 1.25 0)
 			(unlocked yes)
 			(layer "F.SilkS")
@@
 		)
 		(fp_text user "DRV8245"
-			(at -7.337499 -4.064999 270)
+			(at -3.25 0 0)
 			(unlocked yes)
 			(layer "F.SilkS")
@@
 		)
 	)
-	(gr_text "3V3"
-		(at 81.585 74 0)
-		(layer "F.SilkS")
-		(effects
-			(font
-				(size 0.9 0.9)
-				(thickness 0.1)
-			)
-		)
-	)
 	(gr_text "\nUSB_BOOT"
-		(at 85.42 76.07 0)
+		(at 88.5 83 0)
 		(layer "F.SilkS")
 		(effects
@@
 		(min_thickness 0.15)
 		(filled_areas_thickness no)
-		(fill
+		(fill yes
 			(thermal_gap 0.508)
 			(thermal_bridge_width 0.508)
@@
 		(min_thickness 0.15)
 		(filled_areas_thickness no)
-		(fill
+		(fill yes
 			(thermal_gap 0.508)
 			(thermal_bridge_width 0.508)
@@
 		(min_thickness 0.25)
 		(filled_areas_thickness no)
-		(fill
+		(fill yes
 			(thermal_gap 0.5)
 			(thermal_bridge_width 0.5)
@@
 		(min_thickness 0.25)
 		(filled_areas_thickness no)
-		(fill
+		(fill yes
 			(thermal_gap 0.5)
 			(thermal_bridge_width 0.5)
@@
 		(min_thickness 0.2)
 		(filled_areas_thickness no)
-		(fill
+		(fill yes
 			(thermal_gap 0.3)
 			(thermal_bridge_width 0.3)
@@
 		(min_thickness 0.25)
 		(filled_areas_thickness no)
-		(fill
+		(fill yes
 			(thermal_gap 0.5)
 			(thermal_bridge_width 0.5)

Commit message: vault backup: 2025-04-25 06:16:16
Parts:
- added D4: WS2812B, LED_SMD:LED_WS2812B_PLCC4_5.0x5.0mm_P3.2mm, B.Cu at (123.0, 88.2)
- added D7: WS2812B, LED_SMD:LED_WS2812B_PLCC4_5.0x5.0mm_P3.2mm, B.Cu at (108.9, 76.0)
- added D8: WS2812B, LED_SMD:LED_WS2812B_PLCC4_5.0x5.0mm_P3.2mm, B.Cu at (90.7, 76.2)
- added D9: WS2812B, LED_SMD:LED_WS2812B_PLCC4_5.0x5.0mm_P3.2mm, B.Cu at (80.8, 95.5)
Connections:
- J3 pad 13: unconnected-(J3-Pin_13-Pad13) -> +5V
Routing:
- net +5V: track 84.5 -> 195.9 mm, vias 0 -> 1
- net Net-(D8-DOUT): track 0.00 -> 28.6 mm
- net Net-(D7-DOUT): track 0.00 -> 22.3 mm
- net Net-(D4-DOUT): track 0.00 -> 19.4 mm
- net /GPIO23: track 20.9 -> 27.3 mm

Commit message: vault backup: 2025-04-25 06:21:26
Routing:
- net GND: vias 50 -> 79

Commit message: vault backup: 2025-04-25 06:26:33
Routing:
- net +3V3: track 182.9 -> 184.5 mm
- net /GPIO5: track 63.1 -> 63.7 mm
- net /GPIO4: track 63.6 -> 64.2 mm
- net GND: vias 79 -> 60

Commit message: vault backup: 2025-04-25 06:29:06
Routing:
- net GND: vias 60 -> 70
- net +5V: vias 1 -> 2
- net (no net): vias 0 -> 1
Changed lines of the file:
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@@
 		)
 	)
+	(via
+		(at 121 81)
+		(size 0.6)
+		(drill 0.35)
+		(layers "F.Cu" "B.Cu")
+		(net 0)
+	)
 	(segment
 		(start 121.824998 94.462499)
@@
 	)
 	(via
+		(at 75 110)
+		(size 0.6)
+		(drill 0.35)
+		(layers "F.Cu" "B.Cu")
+		(free yes)
+		(net 1)
+	)
+	(via
 		(at 82.75 102)
 		(size 0.6)
@@
 	)
 	(via
+		(at 85.5 74.5)
+		(size 0.6)
+		(drill 0.35)
+		(layers "F.Cu" "B.Cu")
+		(free yes)
+		(net 1)
+	)
+	(via
 		(at 110 109)
 		(size 0.6)
@@
 	)
 	(via
+		(at 73 114)
+		(size 0.6)
+		(drill 0.35)
+		(layers "F.Cu" "B.Cu")
+		(free yes)
+		(net 1)
+	)
+	(via
+		(at 117 102)
+		(size 0.6)
+		(drill 0.35)
+		(layers "F.Cu" "B.Cu")
+		(free yes)
+		(net 1)
+	)
+	(via
 		(at 76.874999 106.375001)
 		(size 0.6)
@@
 	)
 	(via
+		(at 89.5 81)
+		(size 0.6)
+		(drill 0.35)
+		(layers "F.Cu" "B.Cu")
+		(free yes)
+		(net 1)
+	)
+	(via
 		(at 85.75 108)
 		(size 0.6)
@@
 	)
 	(via
+		(at 122 100)
+		(size 0.6)
+		(drill 0.35)
+		(layers "F.Cu" "B.Cu")
+		(free yes)
+		(net 1)
+	)
+	(via
 		(at 97.189994 101.665)
 		(size 0.6)
@@
 	)
 	(via
+		(at 80 121)
+		(size 0.6)
+		(drill 0.35)
+		(layers "F.Cu" "B.Cu")
+		(free yes)
+		(net 1)
+	)
+	(via
 		(at 116 95)
 		(size 0.6)
@@
 	)
 	(via
+		(at 113 83)
+		(size 0.6)
+		(drill 0.35)
+		(layers "F.Cu" "B.Cu")
+		(free yes)
+		(net 1)
+	)
+	(via
 		(at 87.25 81.925)
 		(size 0.6)
@@
 	)
 	(via
+		(at 91 83)
+		(size 0.6)
+		(drill 0.35)
+		(layers "F.Cu" "B.Cu")
+		(free yes)
+		(net 1)
+	)
+	(via
 		(at 105.48 84.96)
 		(size 0.6)
@@
 	)
 	(via
+		(at 80 112)
+		(size 0.6)
+		(drill 0.35)
+		(layers "F.Cu" "B.Cu")
+		(free yes)
+		(net 1)
+	)
+	(via
 		(at 122.824998 94.962499)
 		(size 0.6)
@@
 		(net 65)
 	)
+	(via
+		(at 115 79)
+		(size 0.6)
+		(drill 0.35)
+		(layers "F.Cu" "B.Cu")
+		(net 65)
+	)
 	(segment
 		(start 121.925 85.8)
@@
 		(polygon
 			(pts
-				(xy 140 77) (xy 140 129) (xy 60 129) (xy 60 77)
+				(xy 111.5 77) (xy 111.5 70) (xy 140 70) (xy 140 129) (xy 60 129) (xy 60 77)
 			)
 		)

Commit message: Module Board Done
Parts:
- moved C19 2.00 mm to (84.8, 114.8)
- moved J3 1.50 mm to (108.9, 116.7)
Routing:
- net +5V: track 195.9 -> 198.9 mm
- net VM: track 66.6 -> 63.7 mm
- net /GPIO4: track 64.2 -> 64.8 mm
- net /GPIO5: track 63.7 -> 64.3 mm

Commit message: vault backup: 2025-04-25 21:40:27
Parts:
- added R12: 470, Capacitor_SMD:C_0603_1608Metric_Pad1.08x0.95mm_HandSolder, F.Cu at (104.2, 92.5)
Connections:
- D4 pad 4: /GPIO23 -> GPIO23R
- J4 pad 4: /GPIO23 -> GPIO23R
Routing:
- net /GPIO23: track 27.3 -> 3.87 mm
- net GPIO23R: track 0.00 -> 22.4 mm
- net /GPIO25: track 11.2 -> 12.2 mm
- net /GPIO24: track 18.1 -> 19.0 mm
- net /GPIO26_ADC0: track 13.6 -> 14.2 mm
Other:
- board text added: "0"
- board text added: "1"
- board text added: "23"
- board text added: "24"
- board text added: "25"
- board text added: "26"
- board text added: "27"
- board text added: "28"
- board text added: "29"
- board text added: "3V3"
- board text added: "G"
- board text added: "USB_ BOOT"
- board text removed: "USB_BOOT"
