File: PCBs/ModuleBoard/RP2040_minimal_r2/SwerveModuleBoard.kicad_pcb (KiCad board)
At the start: 2 copper layers, 60 x 52.9 mm, 62 parts, among them IC1 AS5600-ASOT, J1 USB_B_Micro, J2 Conn_02x02_Counter_Clockwise, J3 Conn_02x08_Odd_Even_MountingP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, J4 Conn_01x07, J5 Conn_01x06_Pin, J6 Conn_01x02, J7 Conn_01x06_Pin, U2 W25Q128JVS, U3 RP2040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

Commit message: vault backup: 2025-04-25 21:55:47
Parts:
- moved C21 4.63 mm to (119.4, 103.2), turned to -90 degrees
Routing:
- net VM: track 63.7 -> 70.5 mm
- net GND: track 96.0 -> 93.2 mm, vias 70 -> 74

Commit message: vault backup: 2025-04-25 22:16:16
Parts:
- C19, C21: value 10u -> 100u; footprint Capacitor_SMD:CP_Elec_5x5.4 -> APXE160ARA101MH70G:CAPAE800X700
- moved C21 1.48 mm to (118.0, 103.7)
- moved C19 1.23 mm to (83.6, 115.2)
Routing:
- net GND: track 93.2 -> 78.7 mm, vias 74 -> 79
- net /GPIO5: track 64.3 -> 65.4 mm
- net /GPIO4: track 64.8 -> 65.6 mm

Commit message: vault backup: 2025-04-25 22:21:27
Routing:
- net GND: vias 79 -> 81
- net +5V: vias 2 -> 1
Changed lines of the file:
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@@
 		(tags "capacitor handsolder")
 		(property "Reference" "C20"
-			(at 0.005 -1.5 0)
+			(at -3.25 -0.5 0)
 			(layer "F.SilkS")
 			(effects
@@
 		(tags "DRV8245HQRXZRQ1 ")
 		(property "Reference" "U5"
-			(at -4.537501 0.394857 0)
+			(at -4.537501 2.500001 0)
 			(unlocked yes)
 			(layer "F.SilkS")
@@
 	)
 	(via
+		(at 123 102)
+		(size 0.6)
+		(drill 0.35)
+		(layers "F.Cu" "B.Cu")
+		(free yes)
+		(net 1)
+	)
+	(via
 		(at 107 84.94)
 		(size 0.6)
@@
 	)
 	(via
+		(at 114 80)
+		(size 0.6)
+		(drill 0.35)
+		(layers "F.Cu" "B.Cu")
+		(free yes)
+		(net 1)
+	)
+	(via
 		(at 120 107)
 		(size 0.6)
@@
 	)
 	(segment
-		(start 90.79 116.71)
-		(end 86.326 121.174)
-		(width 0.15)
-		(layer "F.Cu")
-		(net 19)
-	)
-	(segment
-		(start 90.185319 92.676999)
-		(end 90.47099 92.676999)
+		(start 90.769991 92.976)
+		(end 92.551 92.976)
 		(width 0.15)
 		(layer "F.Cu")
@@
 	)
 	(segment
-		(start 72.326 109.855232)
-		(end 72.326 109.8)
+		(start 79 116)
+		(end 72.326 109.326)
 		(width 0.15)
 		(layer "F.Cu")
@@
 	)
 	(segment
-		(start 90.769991 92.976)
-		(end 92.551 92.976)
+		(start 90.47099 92.676999)
+		(end 90.769991 92.976)
 		(width 0.15)
 		(layer "F.Cu")
@@
 	)
 	(segment
-		(start 92.551 92.976)
-		(end 92.625 93.05)
+		(start 77.246388 92.5)
+		(end 77.281742 92.5)
 		(width 0.15)
 		(layer "F.Cu")
@@
 	)
 	(segment
-		(start 76.379168 114.418134)
-		(end 72.326 110.364966)
+		(start 90.08432 92.576)
+		(end 90.185319 92.676999)
 		(width 0.15)
 		(layer "F.Cu")
@@
 	)
 	(segment
-		(start 76.398788 114.418134)
-		(end 76.379168 114.418134)
+		(start 81.874 121.174)
+		(end 79 118.3)
 		(width 0.15)
 		(layer "F.Cu")
@@
 	)
 	(segment
-		(start 72.964645 91.75)
-		(end 76.496388 91.75)
-		(width 0.15)
-		(layer "F.Cu")
-		(net 19)
-	)
-	(segment
-		(start 72.326 110.364966)
-		(end 72.326 109.8)
+		(start 72.326 109.326)
+		(end 72.326 92.388645)
 		(width 0.15)
 		(layer "F.Cu")
@@
 	)
 	(segment
-		(start 81.874 121.174)
-		(end 78.376988 117.676988)
+		(start 77.281742 92.5)
+		(end 77.357742 92.576)
 		(width 0.15)
 		(layer "F.Cu")
@@
 	)
 	(segment
-		(start 91.125 116.71)
-		(end 90.79 116.71)
+		(start 90.79 116.71)
+		(end 86.326 121.174)
 		(width 0.15)
 		(layer "F.Cu")
@@
 	)
 	(segment
-		(start 90.47099 92.676999)
-		(end 90.769991 92.976)
+		(start 86.326 121.174)
+		(end 81.874 121.174)
 		(width 0.15)
 		(layer "F.Cu")
@@
 	)
 	(segment
-		(start 77.281742 92.5)
-		(end 77.357742 92.576)
+		(start 72.964645 91.75)
+		(end 76.496388 91.75)
 		(width 0.15)
 		(layer "F.Cu")
@@
 	)
 	(segment
-		(start 78.376988 116.396334)
-		(end 76.398788 114.418134)
+		(start 90.185319 92.676999)
+		(end 90.47099 92.676999)
 		(width 0.15)
 		(layer "F.Cu")
@@
 	)
 	(segment
-		(start 92.625 93.05)
-		(end 93.0625 93.05)
+		(start 91.125 116.71)
+		(end 90.79 116.71)
 		(width 0.15)
 		(layer "F.Cu")
@@
 	)
 	(segment
-		(start 77.246388 92.5)
-		(end 77.281742 92.5)
+		(start 92.551 92.976)
+		(end 92.625 93.05)
 		(width 0.15)
 		(layer "F.Cu")
@@
 	)
 	(segment
-		(start 86.326 121.174)
-		(end 81.874 121.174)
+		(start 79 118.3)
+		(end 79 116)
 		(width 0.15)
 		(layer "F.Cu")
@@
 	)
 	(segment
-		(start 78.376988 117.676988)
-		(end 78.376988 116.396334)
+		(start 77.357742 92.576)
+		(end 90.08432 92.576)
 		(width 0.15)
 		(layer "F.Cu")
@@
 	)
 	(segment
-		(start 90.08432 92.576)
-		(end 90.185319 92.676999)
+		(start 92.625 93.05)
+		(end 93.0625 93.05)
 		(width 0.15)
 		(layer "F.Cu")
@@
 	)
 	(segment
-		(start 72.326 109.8)
-		(end 72.326 92.388645)
-		(width 0.15)
+		(start 72 92.253612)
+		(end 72.126806 92.126806)
+		(width 0.2)
 		(layer "F.Cu")
-		(net 19)
+		(net 20)
 	)
 	(segment
-		(start 77.357742 92.576)
-		(end 90.08432 92.576)
-		(width 0.15)
+		(start 90.320353 92.350999)
+		(end 90.219354 92.25)
+		(width 0.2)
 		(layer "F.Cu")
-		(net 19)
+		(net 20)
 	)
 	(segment
-		(start 90.320353 92.350999)
-		(end 90.219354 92.25)
+		(start 78.674 116.674)
+		(end 72 110)
 		(width 0.2)
 		(layer "F.Cu")
@@
 	)
 	(segment
-		(start 76.244134 114.744134)
-		(end 76.263754 114.744134)
+		(start 79 118.761034)
+		(end 78.674 118.435034)
 		(width 0.2)
 		(layer "F.Cu")
@@
 	(segment
 		(start 72.854611 91.399)
-		(end 72 92.253611)
+		(end 72.126806 92.126806)
 		(width 0.2)
 		(layer "F.Cu")
@@
 	)
 	(segment
-		(start 72 92.253611)
-		(end 72 110.5)
+		(start 81.6 121.5)
+		(end 79 118.9)
 		(width 0.2)
 		(layer "F.Cu")
@@
 	)
 	(segment
-		(start 88.875 121.5)
-		(end 91.125 119.25)
+		(start 72 110)
+		(end 72 92.253612)
 		(width 0.2)
 		(layer "F.Cu")
@@
 	)
 	(segment
-		(start 72 110.5)
-		(end 76.244134 114.744134)
+		(start 88.875 121.5)
+		(end 81.6 121.5)
 		(width 0.2)
 		(layer "F.Cu")
@@
 	)
 	(segment
-		(start 77.492776 92.25)
-		(end 76.641776 91.399)
+		(start 79 118.9)
+		(end 79 118.761034)
 		(width 0.2)
 		(layer "F.Cu")
@@
 	)
 	(segment
-		(start 81.6 121.5)
-		(end 88.875 121.5)
+		(start 77.492776 92.25)
+		(end 76.641776 91.399)
 		(width 0.2)
 		(layer "F.Cu")
@@
 	)
 	(segment
-		(start 76.263754 114.744134)
-		(end 78.050988 116.531368)
+		(start 91.125 119.25)
+		(end 88.875 121.5)
 		(width 0.2)
 		(layer "F.Cu")
@@
 	)
 	(segment
-		(start 78.050988 116.531368)
-		(end 78.050988 117.950988)
+		(start 72.126806 92.126806)
+		(end 72 92.253611)
 		(width 0.2)
 		(layer "F.Cu")
@@
 	)
 	(segment
-		(start 90.219354 92.25)
-		(end 77.492776 92.25)
+		(start 78.674 118.435034)
+		(end 78.674 116.674)
 		(width 0.2)
 		(layer "F.Cu")
@@
 	)
 	(segment
-		(start 78.050988 117.950988)
-		(end 81.6 121.5)
+		(start 90.219354 92.25)
+		(end 77.492776 92.25)
 		(width 0.2)
 		(layer "F.Cu")
@@
 		(size 0.6)
 		(drill 0.35)
-		(layers "F.Cu" "B.Cu")
-		(net 65)
-	)
-	(via
-		(at 115 79)
-		(size 0.6)
-		(drill 0.35)
