File: PCBs/Main Board/MainBoardPCB/MainBoardPCB.kicad_sch (KiCad schematic)
At the start: 40 parts, among them J1 USB_B_Micro, J3 Conn_02x08_Odd_Even_MountingP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, J4 Conn_01x07, J6 Conn_01x02, J8 Conn_01x06, U1 NCP1117-3.3_SOT223, U2 W25Q128JVS, U3 RP2040, Y1 ABM8-272-T3

Commit message: SO MUCH POWER
Parts:
- added BTSEL2: SW_Push, Button_Switch_THT:SW_PUSH_6mm, symbol Switch:SW_Push
- added C18, C19, C20: 22μF, Capacitor_SMD:C_0603_1608Metric_Pad1.08x0.95mm_HandSolder, symbol Device:C
- added C21: 100 nF, Capacitor_SMD:C_0603_1608Metric_Pad1.08x0.95mm_HandSolder, symbol Device:C
- added C22, C24, C25, C27: 10μF, Capacitor_SMD:C_0603_1608Metric_Pad1.08x0.95mm_HandSolder, symbol Device:C
- added C23, C26: 1nF, Capacitor_SMD:C_0603_1608Metric_Pad1.08x0.95mm_HandSolder, symbol Device:C
- added J5: Conn_01x05, Connector_PinSocket_2.54mm:PinSocket_1x05_P2.54mm_Vertical, symbol Connector_Generic:Conn_01x05
- added L1, L2: 1.5 μH, Capacitor_SMD:C_0603_1608Metric_Pad1.08x0.95mm_HandSolder, symbol Device:L
- added R12: 10k, Resistor_SMD:R_0603_1608Metric_Pad0.98x0.95mm_HandSolder, symbol Device:R
- added R7, R8: 1M, Resistor_SMD:R_0603_1608Metric_Pad0.98x0.95mm_HandSolder, symbol Device:R
- added SW2: 1825910-6, SW4_1825910-B_TEC, symbol Button:1825910-6
- added U4: ESP32-S3-WROOM-1-N16, ESP32-S3-WROOM-1_EXP, symbol 2025-03-19_22-50-46:ESP32-S3-WROOM-1-N16
- added U5, U6: TPS63051RMWR, RMW0012A, symbol TPS63051:TPS63051RMWR
Connections:
- net +3V3: now also C20.2, C21.2, C24.1, C27.1, R12.2, R7.1, R8.1, U4.2 (3V3), U5.4 (VOUT), U5.5 (FB), U6.4 (VOUT), U6.5 (FB)
- net GND: now also BTSEL2.1, C18.1, C19.2, C20.1, C21.1, C22.2, C23.2, C24.2, C25.2, C26.2, C27.2, SW2.3, SW2.4, U4.1 (GND), U4.40 (GND), U4.41 (GND), U4.46 (GND), U4.47 (GND), U4.48 (GND), U4.49 (GND), U5.2 (GND), U5.6 (PWM), U5.9 (GND), U6.2 (GND), U6.6 (PWM), U6.9 (GND)
- net VBUS: no longer names the net of C1.1, J1.1 (VBUS), U1.3 (VI)
- new net: L1.1, U5.1 (L1)
- new net: L1.2, U5.3 (L2)
- new net: R7.2, U5.8 (PG)
- new net: BTSEL2.2, C18.2, C19.1, R12.1, U4.3 (EN)
- new net: L2.1, U6.1 (L1)
- new net: L2.2, U6.3 (L2)
- new net: SW2.1, SW2.2, U4.27 (IO0)
- new net: C26.1, U6.7 (SS)
- new net: J5.5 (Pin_5), U4.15 (IO3)
- new net: J5.4 (Pin_4), U4.16 (IO46)
- new net: J5.3 (Pin_3), U4.17 (IO9)
- new net: J5.2 (Pin_2), U4.18 (IO10)
- new net: J5.1 (Pin_1), U4.19 (IO11)
- new net: R8.2, U6.8 (PG)
- new net: C23.1, U5.7 (SS)
- new net D+: U4.14 (IO20)
- new net D-: U4.13 (IO19)
- new net IMU_CS: U4.9 (IO16)
- new net IMU_SCLK: U4.12 (IO8)
- new net IMU_SDI: U4.11 (IO18)
- new net IMU_SDO: U4.10 (IO17)
- new net LED_1: U4.32 (IO39)
- new net LED_2: U4.33 (IO40)
- new net LED_3: U4.34 (IO41)
- new net LED_4: U4.35 (IO42)
- new net Motor_1_PWM: U4.28 (IO35)
- new net Motor_2_PWM: U4.29 (IO36)
- new net Motor_3_PWM: U4.30 (IO37)
- new net Motor_4_PWM: U4.31 (IO38)
- new net VAA: C22.1, C25.1, U5.11 (EN), U5.12 (VIN), U6.11 (EN), U6.12 (VIN)
Other:
- note added: "Connectors"
- note removed: "Main Connector"
- moved on the sheet: C1, C4, D1, D2, J1, J3, J6, R10, R11, U1

Commit message: AH BOARDS
Parts:
- removed L1, L2: 1.5 μH, Capacitor_SMD:C_0603_1608Metric_Pad1.08x0.95mm_HandSolder, symbol Device:L
- removed U1: NCP1117-3.3_SOT223, Package_TO_SOT_SMD:SOT-223-3_TabPin2, symbol Regulator_Linear:NCP1117-3.3_SOT223
- removed U5, U6: TPS63051RMWR, RMW0012A, symbol TPS63051:TPS63051RMWR
- added C28, C29, C30, C31, C32, C33: 22 uF, Capacitor_SMD:C_1206_3216Metric_Pad1.33x1.80mm_HandSolder, symbol Device:C
- added D3, D4: PMEG3020EXEX, Diode_SMD:D_SOD-123F, symbol Device:D
- added J2: USB4105-GF-A, USB4105_GF_A(2):GCT_USB4105-GF-A, symbol USB4105-GF-A:USB4105-GF-A
- added R13, R14, R6: 10k, Resistor_SMD:R_0603_1608Metric, symbol Device:R
- added R9: 5.1k, Resistor_SMD:R_0603_1608Metric_Pad0.98x0.95mm_HandSolder, symbol Device:R
- added TP5, TP6: TestPoint, Connector_Pin:Pin_D1.0mm_L10.0mm, symbol Connector:TestPoint
- added U1: TPS566238PRQFR, RQF0009A, symbol TPS556:TPS566238PRQFR
- added U5, U6: MIC5219-3.3YM5, Package_TO_SOT_SMD:SOT-23-5, symbol Regulator_Linear:MIC5219-3.3YM5
- C22: value 10μF -> 470 pF; footprint Capacitor_SMD:C_0603_1608Metric_Pad1.08x0.95mm_HandSolder -> Capacitor_SMD:C_0603_1608Metric
- C23, C26: value 1nF -> 22 uF; footprint Capacitor_SMD:C_0603_1608Metric_Pad1.08x0.95mm_HandSolder -> Capacitor_SMD:C_1206_3216Metric_Pad1.33x1.80mm_HandSolder
- C24, C27: value 10μF -> 22 uF; footprint Capacitor_SMD:C_0603_1608Metric_Pad1.08x0.95mm_HandSolder -> Capacitor_SMD:C_1206_3216Metric_Pad1.33x1.80mm_HandSolder
- C25: value 10μF -> 10u
- C4: value 10u -> 470 pF; footprint Capacitor_SMD:C_0603_1608Metric_Pad1.08x0.95mm_HandSolder -> Capacitor_SMD:C_0603_1608Metric
- R7: value 1M -> 10k; footprint Resistor_SMD:R_0603_1608Metric_Pad0.98x0.95mm_HandSolder -> Resistor_SMD:R_0603_1608Metric
- R8: value 1M -> 5.1k
Connections:
- net +3V3: now also C23.1, U5.5 (OUT), U6.5 (OUT); no longer C27.1, C4.1, R7.1, R8.1
- net D+: now also J2.A6 (DP1), J2.B6 (DP2), TP5.1
- net D-: now also J2.A7 (DN1), J2.B7 (DN2), TP6.1
- net GND: now also R8.2, J2.A1_B12 (GND), J2.B1_A12 (GND__1), J2.SH1 (SHELL_GND), J2.SH2 (SHELL_GND__1), J2.SH3 (SHELL_GND__2), J2.SH4 (SHELL_GND__3), R9.1, U5.2 (GND), U6.2 (GND); no longer C26.2, C27.2
- net VAA: now also C26.1, C27.1; no longer C22.1, C25.1
- net VUSB: now reaches C1.1, J1.1 (VBUS)
- net VUSB: now also C25.1, D3.2 (A), J2.A4_B9 (VBUS), J2.B4_A9 (VBUS__1)
- net at R7.2: now also U6.3 (EN)
- new net: D3.1 (K), D4.1 (K), R6.1, R7.1, U5.1 (IN), U6.1 (IN)
- new net: C26.2, C27.2, U1.5 (VIN), U1.6 (VIN)
- new net: J2.A5 (CC1), R9.2
- new net: C22.1, U5.4 (BP)
- new net: C29.1, U1.9 (SS)
- new net: C31.2, R13.1, U1.2 (FB)
- new net: R6.2, U5.3 (EN)
- new net: C4.1, U6.4 (BP)
- new net: C28.1, U1.1 (VCC)
- new net: C30.1, U1.7 (BST)
- new net: C30.2, U1.8 (SW)
- new net: J2.B5 (CC2), R8.1
- new net +5V: D4.2 (A)
Other:
- moved on the sheet: C1, J1
