File: PCBs/Main Board/MainBoardPCB/MainBoardPCB.kicad_pcb (KiCad board)
At the start: 4 copper layers, 56 x 74 mm, 87 parts, among them J1 USB_B_Micro, J2 USB_B_Micro, J3 Conn_02x08_Odd_Even_MountingP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, J4 Conn_02x08_Odd_Even_MountingP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, J5 Conn_01x02, J6 Conn_01x02, J7 Conn_01x03, J8 Conn_01x03, J9 Conn_02x05_Counter_Clockwise, U1 TPS566238PRQFR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

Commit message: Goofy
Other:
- board text added: "WPI"
