File: PCBs/Main Board/MainBoardPCB/MainBoardPCB.kicad_pcb (KiCad board)
At the start: 2 copper layers, 56 x 84 mm, 37 parts, among them J3 Conn_02x08_Odd_Even_MountingP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, J4 Conn_01x07, J6 Conn_01x02, J8 Conn_01x06, U1 NCP1117-3.3_SOT223, Y1 ABM8-272-T3

Commit message: vault backup: 2025-04-24 15:59:31
Parts:
- moved J3 19.3 mm to (42.5, 42.3)
Changed lines of the file:
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@@
 	(footprint "Connector_PinHeader_2.54mm:PinHeader_2x08_P2.54mm_Vertical"
 		(layer "F.Cu")
-		(at 61.42 38.55)
+		(at 42.46 42.3)
 		(descr "Through hole straight pin header, 2x08, 2.54mm pitch, double rows")
 		(tags "Through hole pin header THT 2x08 2.54mm double row")

Commit message: vault backup: 2025-04-24 16:00:18
Parts:
- moved H1 0.51 mm to (56.0, 25.0)
Other:
- board size 56 x 84 mm -> 56 x 74 mm
Changed lines of the file:
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@@
 	(footprint "MountingHole:MountingHole_3.2mm_M3_DIN965_Pad_TopBottom"
 		(layer "F.Cu")
-		(at 55.55 24.77)
+		(at 56 25)
 		(descr "Mounting Hole 3.2mm, M3, DIN965")
 		(tags "mounting hole 3.2mm m3 din965")
@@
 		)
 	)
+	(gr_line
+		(start 96.535533 41)
+		(end 96.535534 41)
+		(stroke
+			(width 0.2)
+			(type default)
+		)
+		(layer "Edge.Cuts")
+	)
 	(gr_arc
-		(start 92 35.303061)
-		(mid 94.872983 37.039763)
-		(end 95.999999 40.20204)
+		(start 92.535534 36.101021)
+		(mid 89.66255 34.364319)
+		(end 88.535534 31.181752)
 		(stroke
 			(width 0.2)
@@
 		(layer "Edge.Cuts")
 	)
-	(gr_line
-		(start 40 40)
-		(end 40 62.202042)
+	(gr_arc
+		(start 44.535534 67.898979)
+		(mid 41.66255 66.162278)
+		(end 40.535534 63.000002)
 		(stroke
 			(width 0.2)
@@
 	)
 	(gr_arc
-		(start 40 40)
-		(mid 41.127017 36.837722)
-		(end 44 35.101019)
+		(start 92.535534 36.101021)
+		(mid 95.408517 37.837723)
+		(end 96.535533 41)
 		(stroke
 			(width 0.2)
@@
 	)
 	(gr_arc
-		(start 88 83.20204)
-		(mid 68 103.20204)
-		(end 48 83.20204)
+		(start 83.535534 20)
+		(mid 87.071068 21.464466)
+		(end 88.535534 25)
 		(stroke
 			(width 0.2)
@@
 		(layer "Edge.Cuts")
 	)
-	(gr_line
-		(start 88 83.20204)
-		(end 88 72.20204)
+	(gr_arc
+		(start 88.535534 89)
+		(mid 87.071068 92.535534)
+		(end 83.535534 94)
 		(stroke
 			(width 0.2)
@@
 	)
 	(gr_line
-		(start 88 30.383792)
-		(end 88 24.20204)
+		(start 88.535534 89)
+		(end 88.535534 73)
 		(stroke
 			(width 0.2)
@@
 		(layer "Edge.Cuts")
 	)
-	(gr_arc
-		(start 96 62.40408)
-		(mid 94.872983 65.566358)
-		(end 92 67.303061)
+	(gr_line
+		(start 48.535534 25)
+		(end 48.535534 30.999998)
 		(stroke
 			(width 0.2)
@@
 	)
 	(gr_arc
-		(start 48 30.202038)
-		(mid 46.872983 33.364317)
-		(end 44 35.101019)
+		(start 88.535534 73)
+		(mid 89.662551 69.837722)
+		(end 92.535534 68.101021)
 		(stroke
 			(width 0.2)
@@
 	)
 	(gr_line
-		(start 48 71.999997)
-		(end 48 83.20204)
+		(start 83.535534 20)
+		(end 53.535533 20)
 		(stroke
 			(width 0.2)
@@
 		(layer "Edge.Cuts")
 	)
-	(gr_arc
-		(start 83 19.20204)
-		(mid 86.535534 20.666506)
-		(end 88 24.20204)
+	(gr_line
+		(start 96.535534 63.20204)
+		(end 96.535534 41)
 		(stroke
 			(width 0.2)
@@
 	)
 	(gr_arc
-		(start 92 35.303061)
-		(mid 89.127016 33.566359)
-		(end 88 30.383792)
+		(start 48.535534 30.999998)
+		(mid 47.408517 34.162277)
+		(end 44.535534 35.898979)
 		(stroke
 			(width 0.2)
@@
 	)
 	(gr_line
-		(start 95.999999 40.20204)
-		(end 96 40.20204)
+		(start 53.535534 94)
+		(end 83.535534 94)
 		(stroke
 			(width 0.2)
@@
 		(layer "Edge.Cuts")
 	)
-	(gr_line
-		(start 83 19.20204)
-		(end 52.999999 19.20204)
+	(gr_arc
+		(start 53.535534 94)
+		(mid 50 92.535534)
+		(end 48.535534 89.000001)
+		(stroke
+			(width 0.2)
+			(type default)
+		)
+		(layer "Edge.Cuts")
+	)
+	(gr_arc
+		(start 44.535534 67.898979)
+		(mid 47.408518 69.635681)
+		(end 48.535534 72.797957)
 		(stroke
 			(width 0.2)
@@
 	)
 	(gr_line
-		(start 96 62.40408)
-		(end 96 40.20204)
+		(start 48.535534 72.797957)
+		(end 48.535534 89.000001)
 		(stroke
 			(width 0.2)
@@
 	)
 	(gr_arc
-		(start 48 24.202041)
-		(mid 49.464466 20.666506)
-		(end 52.999999 19.20204)
+		(start 96.535534 63.20204)
+		(mid 95.408517 66.364318)
+		(end 92.535534 68.101021)
 		(stroke
 			(width 0.2)
@@
 		(layer "Edge.Cuts")
 	)
-	(gr_arc
-		(start 88 72.20204)
-		(mid 89.127017 69.039762)
-		(end 92 67.303061)
+	(gr_line
+		(start 88.535534 31.181752)
+		(end 88.535534 25)
 		(stroke
 			(width 0.2)
@@
 	)
 	(gr_arc
-		(start 44 67.101019)
-		(mid 41.127016 65.364318)
-		(end 40 62.202042)
+		(start 48.535534 25)
+		(mid 50 21.464466)
+		(end 53.535533 20)
 		(stroke
 			(width 0.2)
@@
 		(layer "Edge.Cuts")
 	)
-	(gr_line
-		(start 48 24.202041)
-		(end 48 30.202038)
+	(gr_arc
+		(start 40.535534 40.79796)
+		(mid 41.662551 37.635682)
+		(end 44.535534 35.898979)
 		(stroke
 			(width 0.2)
@@
 		(layer "Edge.Cuts")
 	)
-	(gr_arc
-		(start 44 67.101019)
-		(mid 46.872984 68.837721)
-		(end 48 71.999997)
+	(gr_line
+		(start 40.535534 40.79796)
+		(end 40.535534 63.000002)
 		(stroke
 			(width 0.2)
@@
 	)
 	(group ""
-		(members "01454156-cbf1-4c60-9d7f-f4e73c28cb71" "0330eccb-6d07-4053-9667-dbec7af50e90"
-			"085e94e7-7aa8-46bb-b2e2-de18433473f6" "14fd1893-15d3-4d50-bdd7-3c05ab350c7a"
-			"1d5b0817-93af-4b92-9083-141c31520433" "2320bfd8-3e29-44be-85b2-2b3fd8af9ece"
-			"26f60caa-3642-4267-99f4-38db80fbbec2" "2c8991b4-bf5d-49e3-8ddd-dc48b790fe5d"
-			"3ed1322c-1c06-40b0-8da2-2c3323ed668f" "483bc9ae-4def-492c-b2e7-4f654d9c0f81"
-			"4ffbd0f7-88f2-4d95-96da-92cbe7ae9d7b" "8096124f-feb1-4ca2-a6ac-b3400a7bd6c4"
-			"9ead0c6f-607e-45ee-aeca-eb2a745409c1" "a6670fcc-d5c4-4fd4-9a93-5d2cfe212b65"
-			"b550e110-abbc-453f-9979-6c75e094b8da" "c823120d-0fe9-4406-9b62-1ba66bf8073b"
-			"c8cadf6a-9aeb-4983-851d-097e5c0c3f07" "d0c33aa0-7bc7-43cd-a982-a94c12a239b8"
-			"f8e80ca7-08a2-4ff5-81d9-dd3bb462bc07"
+		(members "0f7f4629-b028-4f7a-8961-3516cf0bd3dc" "139e9e1f-ac28-4462-a8f0-3a2831b8170b"
+			"297c2a93-2b45-40b0-9b2c-396e771f42e9" "4a141715-77e8-4204-b9f4-91360282721f"
+			"4e983614-c636-42ba-807a-4a7dbab2e7a0" "510bd445-07e3-49ab-adcf-e04acc0ac152"
+			"5cd59799-f268-43f1-bb03-b73cfa04fab3" "5f327820-d8a1-4651-967b-16692802ab58"
+			"6cb1fade-8d05-4aaf-bead-3a90d41cbd0c" "7725aed6-d275-4b24-9e99-82d77d2e2761"
+			"7ed6d7b7-4dc2-45c7-82b4-afa62b8a272b" "83c9c3ac-9356-4d85-b7f0-305de5b16c7e"
+			"afa54840-dbcd-4bc5-a4ef-414a8a678195" "b2a691b9-47b1-41be-8752-2ab5c90438b4"
+			"ca61e5c0-ebd3-417d-bf6b-3c00d07331c5" "d191e12f-8a6e-4bb7-8801-b6372c80d5d3"
+			"d73edba7-8ac6-464d-b6aa-f407f112fdd4" "e190d88d-884c-4507-b820-16bc1e5cdc41"
+			"e38147f0-0668-45c1-8644-b264b0f957cd" "eb5d821a-d2d9-454b-ac22-0e6dda32f52b"
+			"f57ddb6e-dce9-47e2-ad1b-2976e4cd9eff"
 		)
 	)

Commit message: board go brrr
Parts:
- added BTSEL2: SW_Push, Button_Switch_THT:SW_PUSH_1P1T_6x3.5mm_H5.0_APEM_MJTP1250, F.Cu at (82.0, 55.7)
- added BTSEL3: SW_Push, Button_Switch_THT:SW_PUSH_1P1T_6x3.5mm_H5.0_APEM_MJTP1250, F.Cu at (79.3, 91.9)
- added C18: 22μF, Capacitor_SMD:C_0402_1005Metric_Pad0.74x0.62mm_HandSolder, F.Cu at (78.9, 53.0)
- added C19: 22μF, Capacitor_SMD:C_0402_1005Metric_Pad0.74x0.62mm_HandSolder, F.Cu at (67.3, 70.6)
- added C20: 22μF, Capacitor_SMD:C_0402_1005Metric_Pad0.74x0.62mm_HandSolder, F.Cu at (66.7, 66.6)
- added C21: 100 nF, Capacitor_SMD:C_0402_1005Metric_Pad0.74x0.62mm_HandSolder, F.Cu at (67.8, 66.6)
- added C22: 470 pF, Capacitor_SMD:C_0402_1005Metric_Pad0.74x0.62mm_HandSolder, F.Cu at (62.1, 85.4)
- added C23: 22 uF, Capacitor_SMD:C_0603_1608Metric_Pad1.08x0.95mm_HandSolder, F.Cu at (65.0, 82.9)
- added C24: 22 uF, Capacitor_SMD:C_0603_1608Metric_Pad1.08x0.95mm_HandSolder, F.Cu at (65.0, 79.3)
- added C25: 10u, Capacitor_SMD:C_0402_1005Metric_Pad0.74x0.62mm_HandSolder, F.Cu at (69.0, 86.2)
- added C26: 100 nF, Capacitor_SMD:C_0402_1005Metric_Pad0.74x0.62mm_HandSolder, F.Cu at (51.7, 41.6)
- added C27: 47 uF, Capacitor_SMD:C_0603_1608Metric_Pad1.08x0.95mm_HandSolder, F.Cu at (51.3, 40.0)
- added C28: 1 uF, Capacitor_SMD:C_0402_1005Metric_Pad0.74x0.62mm_HandSolder, F.Cu at (56.6, 43.1)
- added C29: 10 nF, Capacitor_SMD:C_0402_1005Metric_Pad0.74x0.62mm_HandSolder, F.Cu at (54.6, 43.4)
- added C30: 100 nF, Capacitor_SMD:C_0402_1005Metric_Pad0.74x0.62mm_HandSolder, F.Cu at (52.7, 43.0)
- added C31: 33 pF, Capacitor_SMD:C_0402_1005Metric_Pad0.74x0.62mm_HandSolder, F.Cu at (57.8, 41.4)
- added C32: 22 uF, Capacitor_SMD:C_0603_1608Metric_Pad1.08x0.95mm_HandSolder, F.Cu at (54.1, 54.1)
- added C33: 100 nF, Capacitor_SMD:C_0402_1005Metric_Pad0.74x0.62mm_HandSolder, F.Cu at (54.0, 55.6)
- added C34: 22 uF, Capacitor_SMD:C_0603_1608Metric_Pad1.08x0.95mm_HandSolder, F.Cu at (71.4, 52.5)
- added D3: PMEG3020EXEX, Diode_SMD:D_SOD-123F, F.Cu at (67.0, 85.2)
- added D4: PMEG3020EXEX, Diode_SMD:D_SOD-123F, F.Cu at (54.5, 83.6)
- added J1: USB_B_Micro, Connector_USB:USB_Micro-B_Amphenol_10103594-0001LF_Horizontal, F.Cu at (70.7, 90.4)
- added J2: USB_B_Micro, Connector_USB:USB_Micro-B_Amphenol_10103594-0001LF_Horizontal, F.Cu at (61.0, 90.4)
- added J5: Conn_01x02, Connector_JST:JST_EH_B2B-EH-A_1x02_P2.50mm_Vertical, F.Cu at (76.5, 34.0)
- added J7: Conn_01x03, Connector_JST:JST_EH_B3B-EH-A_1x03_P2.50mm_Vertical, F.Cu at (75.5, 40.0)
- added L1: L, Library:IND_SPM6530_TDK, F.Cu at (54.4, 49.1)
- added R12: 10k, Resistor_SMD:R_0402_1005Metric_Pad0.72x0.64mm_HandSolder, F.Cu at (67.3, 68.9)
- added R13: 220k, Resistor_SMD:R_0402_1005Metric_Pad0.72x0.64mm_HandSolder, F.Cu at (56.7, 41.4)
- added R14: 30k, Resistor_SMD:R_0402_1005Metric_Pad0.72x0.64mm_HandSolder, F.Cu at (56.7, 39.0)
- added R6: 10k, Resistor_SMD:R_0402_1005Metric_Pad0.72x0.64mm_HandSolder, F.Cu at (59.4, 83.1)
- added R7: 10k, Resistor_SMD:R_0402_1005Metric_Pad0.72x0.64mm_HandSolder, F.Cu at (59.3, 79.3)
- added R8: 100k, Resistor_SMD:R_0402_1005Metric_Pad0.72x0.64mm_HandSolder, F.Cu at (59.9, 38.2)
- added R9: 20k, Resistor_SMD:R_0402_1005Metric_Pad0.72x0.64mm_HandSolder, F.Cu at (59.9, 40.6)
- added U2: W25Q128JVS, MainBoard:SOIC_128JVSIQ_WIN, F.Cu at (51.8, 62.2)
- added U3: RP2040, Package_DFN_QFN:QFN-56-1EP_7x7mm_P0.4mm_EP3.2x3.2mm_ThermalVias, F.Cu at (56.5, 70.7)
- added U4: ESP32-S3-WROOM-1-N16, MainBoard:ESP32-S3-WROOM-1_EXP, F.Cu at (78.2, 71.1)
- added U5: MIC5219-3.3YM5, MainBoard:MIC, F.Cu at (62.1, 83.0)
- added U6: MIC5219-3.3YM5, MainBoard:MIC, F.Cu at (62.1, 79.2)
- added U7: LSM6DSVTR, MainBoard:LGA14-L_2P59X3P1X0P5_STM, F.Cu at (68.5, 52.0)
- BTSEL1: footprint Button_Switch_THT:SW_PUSH_6mm -> Button_Switch_THT:SW_PUSH_1P1T_6x3.5mm_H5.0_APEM_MJTP1250
- C1, C10, C11, C12, C13, C14, C15, C16, C17, C2, C3, C5, C6, C7, C8, C9: footprint Capacitor_SMD:C_0603_1608Metric_Pad1.08x0.95mm_HandSolder -> Capacitor_SMD:C_0402_1005Metric_Pad0.74x0.62mm_HandSolder
- C4: value 10u -> 470 pF; footprint Capacitor_SMD:C_0603_1608Metric_Pad1.08x0.95mm_HandSolder -> Capacitor_SMD:C_0402_1005Metric_Pad0.74x0.62mm_HandSolder
- J4: value Conn_01x07 -> Conn_02x08_Odd_Even_MountingPin; footprint Connector_PinSocket_2.54mm:PinSocket_1x07_P2.54mm_Vertical -> Connector_PinHeader_2.54mm:PinHeader_2x08_P2.54mm_Vertical
- J8: value Conn_01x06 -> Conn_01x03; footprint Connector_PinHeader_2.54mm:PinHeader_1x06_P2.54mm_Vertical -> Connector_JST:JST_EH_B3B-EH-A_1x03_P2.50mm_Vertical
- R1, R10, R11, R2, R3, R4, R5: footprint Resistor_SMD:R_0603_1608Metric_Pad0.98x0.95mm_HandSolder -> Resistor_SMD:R_0402_1005Metric_Pad0.72x0.64mm_HandSolder
- U1: value NCP1117-3.3_SOT223 -> TPS566238PRQFR; footprint Package_TO_SOT_SMD:SOT-223-3_TabPin2 -> MainBoard:RQF0009A
- moved C1 63.5 mm to (64.0, 85.9), turned to 90 degrees
- moved H3 57.2 mm to (83.5, 89.0)
- moved C13 54.7 mm to (64.4, 76.8)
- moved C3 53.4 mm to (57.7, 80.7), turned to -90 degrees
- moved C7 53.3 mm to (59.2, 75.3)
- moved Y1 52.2 mm to (55.4, 78.3), turned to -90 degrees
- moved R5 51.2 mm to (57.7, 78.4), turned to -90 degrees
- moved C2 51.0 mm to (55.4, 75.6), turned to 180 degrees
- moved C14 50.0 mm to (64.5, 74.7)
- moved C9 48.3 mm to (64.5, 75.7)
- moved C4 46.8 mm to (62.1, 76.8), turned to 180 degrees
- moved C15 46.6 mm to (64.5, 73.8)
- moved C16 44.4 mm to (62.1, 73.7), turned to 180 degrees
- moved R3 43.4 mm to (58.0, 65.1), turned to -90 degrees
- moved H4 42.8 mm to (53.5, 89.0)
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Connections:
- C1 pad 1: VBUS -> VUSB
- C4 pad 1: +3V3 -> Net-(U6-BP)
- D1 pad 2: /GPIO21 -> LED2
- D2 pad 2: /GPIO22 -> LED1
- J3 pad 1: VM -> VAA
- J3 pad 13: unconnected-(J3-Pin_13-Pad13) -> +5V
- J3 pad 14: unconnected-(J3-Pin_14-Pad14) -> +5V
- J3 pad 2: VM -> VAA
- J3 pad 3: VM -> VAA
- J3 pad 4: VM -> VAA
- J3 pad 5: VM -> VAA
- J3 pad 6: VM -> VAA
- J4 pad 1: /GPIO23 -> VAA
- J4 pad 2: /GPIO24 -> VAA
- J4 pad 3: /GPIO25 -> VAA
- J4 pad 4: /GPIO26_ADC0 -> VAA
- J4 pad 5: /GPIO27_ADC1 -> VAA
- J4 pad 6: /GPIO28_ADC2 -> VAA
- J4 pad 7: /GPIO29_ADC3 -> GND
- J6 pad 2: VM -> VAA
- J8 pad 1: /GPIO0 -> GND
- J8 pad 2: /GPIO1 -> +5V
- J8 pad 3: /GPIO2 -> Servo2
- U1 pad 1: GND -> Net-(U1-VCC)
- U1 pad 2: +3V3 -> Net-(U1-FB)
- U1 pad 3: VBUS -> unconnected-(U1-EN-Pad3)
Routing:
- net +5V: track 0.00 -> 109.7 mm, vias 0 -> 4
- net VAA: track 0.00 -> 95.9 mm, vias 0 -> 37
- net /GPIO5: track 0.00 -> 79.4 mm, vias 0 -> 2
- net /GPIO4: track 0.00 -> 71.6 mm, vias 0 -> 2
- net +3V3: track 0.00 -> 68.1 mm, vias 0 -> 12
- net RX: track 0.00 -> 45.3 mm, vias 0 -> 1
- net Servo2: track 0.00 -> 36.7 mm, vias 0 -> 1
- net Servo1: track 0.00 -> 36.1 mm, vias 0 -> 3
- net /USB_D+: track 0.00 -> 34.2 mm
- net BATT_READ: track 0.00 -> 33.6 mm, vias 0 -> 2
- net /USB_D-: track 0.00 -> 31.3 mm
- net Net-(U4-EN): track 0.00 -> 30.5 mm
- net +1V1: track 0.00 -> 21.3 mm, vias 0 -> 4
- net GYROSDA: track 0.00 -> 21.2 mm, vias 0 -> 2
- net GYROSCL: track 0.00 -> 21.2 mm, vias 0 -> 2
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- added copper zone on B.Cu, net +3V3
- added copper zone on F.Cu, net +3V3
- added copper zone on B.Cu, net GND
- added copper zone on F.Cu, net GND
- added copper zone on In1.Cu, net GND
- added copper zone on In2.Cu, net GND
- added copper zone on F.Cu, net Net-(U1-FB)
- added copper zone on F.Cu, net Net-(U1-SW)
- added copper zone on B.Cu, net VAA
- added copper zone on F.Cu, net VAA
Other:
- copper layers 2 -> 4

Commit message: Go us
Parts:
- added D5: LED, LED_SMD:LED_0603_1608Metric_Pad1.05x0.95mm_HandSolder, F.Cu at (49.6, 74.0)
- added D6: LED, LED_SMD:LED_0603_1608Metric_Pad1.05x0.95mm_HandSolder, F.Cu at (51.2, 74.0)
- added D7: LED, LED_SMD:LED_0603_1608Metric_Pad1.05x0.95mm_HandSolder, F.Cu at (49.8, 79.9)
- added D8: LED, LED_SMD:LED_0603_1608Metric_Pad1.05x0.95mm_HandSolder, F.Cu at (51.5, 79.9)
- added J9: Conn_02x05_Counter_Clockwise, Connector_PinHeader_2.54mm:PinHeader_2x05_P2.54mm_Vertical, F.Cu at (73.5, 23.5)
- added R15: 10k, Resistor_SMD:R_0402_1005Metric_Pad0.72x0.64mm_HandSolder, F.Cu at (66.3, 53.8)
- added R16: 10k, Resistor_SMD:R_0402_1005Metric_Pad0.72x0.64mm_HandSolder, F.Cu at (65.7, 52.0)
- added R17: 430, Resistor_SMD:R_0402_1005Metric_Pad0.72x0.64mm_HandSolder, F.Cu at (49.5, 77.0)
- added R18: 430, Resistor_SMD:R_0402_1005Metric_Pad0.72x0.64mm_HandSolder, F.Cu at (51.1, 76.9)
- added R19: 430, Resistor_SMD:R_0402_1005Metric_Pad0.72x0.64mm_HandSolder, F.Cu at (49.4, 82.9)
- added R20: 430, Resistor_SMD:R_0402_1005Metric_Pad0.72x0.64mm_HandSolder, F.Cu at (53.5, 81.2)
- D3, D4: footprint Diode_SMD:D_SOD-123F -> Diode_SMD:D_SOD-128
- moved C25 1.98 mm to (71.0, 85.9)
- moved C1 1.69 mm to (62.7, 87.0), turned to 180 degrees
- moved D3 0.82 mm to (67.2, 86.0), turned to 0 degrees
- moved C23 0.49 mm to (65.0, 82.4)
- moved C24 0.35 mm to (65.0, 79.0)
Connections:
- U3 pad 11: /GPIO8 -> LED3
- U3 pad 12: /GPIO9 -> LED4
- U3 pad 13: /GPIO10 -> LED5
- U3 pad 14: /GPIO11 -> LED6
- U3 pad 36: /GPIO24 -> 2040TX
- U3 pad 37: /GPIO25 -> 2040RX
- U4 pad 10: IMU_SDO -> unconnected-(U4-IO17-Pad10)
- U4 pad 11: IMU_SDI -> unconnected-(U4-IO18-Pad11)
- U4 pad 12: IMU_SCLK -> unconnected-(U4-IO8-Pad12)
- U4 pad 28: Motor_1_PWM -> unconnected-(U4-IO35-Pad28)
- U4 pad 29: Motor_2_PWM -> unconnected-(U4-IO36-Pad29)
- U4 pad 30: Motor_3_PWM -> Net-(J9-Pin_6)
- U4 pad 31: Motor_4_PWM -> Net-(J9-Pin_5)
- U4 pad 32: LED_1 -> Net-(J9-Pin_4)
- U4 pad 33: LED_2 -> Net-(J9-Pin_3)
- U4 pad 34: LED_3 -> Net-(J9-Pin_2)
- U4 pad 35: LED_4 -> Net-(J9-Pin_1)
- U4 pad 6: unconnected-(U4-IO6-Pad6) -> 2040RX
- U4 pad 7: unconnected-(U4-IO7-Pad7) -> 2040TX
- U4 pad 9: IMU_CS -> unconnected-(U4-IO16-Pad9)
- U7 pad 1: unconnected-(U7-SDO/SA0-Pad1) -> GND
- U7 pad 10: unconnected-(U7-OCS_AUX-Pad10) -> GND
- U7 pad 11: unconnected-(U7-SDO_AUX-Pad11) -> GND
- U7 pad 12: unconnected-(U7-CS-Pad12) -> +3V3
- U7 pad 13: GYROSCL -> Net-(U7-SCL)
- U7 pad 14: GYROSDA -> Net-(U7-SDA)
Routing:
- net Net-(J9-Pin_5): track 0.00 -> 67.0 mm, vias 0 -> 1
- net Net-(J9-Pin_6): track 0.00 -> 66.2 mm, vias 0 -> 1
- net Net-(J9-Pin_3): track 0.00 -> 62.0 mm, vias 0 -> 1
- net Net-(J9-Pin_4): track 0.00 -> 61.7 mm, vias 0 -> 1
- net Net-(J9-Pin_1): track 0.00 -> 57.9 mm, vias 0 -> 1
- net Net-(J9-Pin_2): track 0.00 -> 57.6 mm, vias 0 -> 2
- net +3V3: track 68.1 -> 103.0 mm, vias 12 -> 10
- net +5V: track 109.7 -> 141.0 mm
- net 2040TX: track 0.00 -> 10.7 mm, vias 0 -> 2
- net 2040RX: track 0.00 -> 10.5 mm, vias 0 -> 2
- net LED5: track 0.00 -> 8.26 mm
- net LED6: track 0.00 -> 6.37 mm
- net /USB_D+: track 34.2 -> 39.5 mm, vias 0 -> 2
- net Servo2: track 36.7 -> 31.5 mm
- net VUSB: track 14.8 -> 19.8 mm
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